Commit message: Arruma posição e orientação das cameras do ros Inverte/Arruma nome das cameras da direita/esquerda

File: urdf/fsr_husky_parts/pointgrey_flea3.urdf.xacro (robot description, xacro)
@@ -112,5 +112,5 @@
 			<parent link="${prefix}_camera_standoff"/>
 			<child link="${prefix}_camera"/>
-			<origin xyz="0 0 ${standoff_length/2+flea_size/2}" rpy="${camera_r} ${1.5708+camera_p} ${camera_y}" />
+			<origin xyz="0 0 ${standoff_length/2+flea_size/2}" rpy="${camera_r} ${camera_p} ${camera_y}" />
 		</joint>
 		<!-- Camera Lense -->
@@ -121,5 +121,5 @@
         				<cylinder length="${lense_length}" radius="${lense_radius}"/>
       				</geometry>
-				<origin rpy="0 0 0" xyz="0 0 0"/>
+				<origin rpy="0 1.57 0" xyz="0 0 -0.035"/>
       				<material name="Black"/>
     			</visual>

File: urdf/husky.urdf.xacro (robot description, xacro)
@@ -185,6 +185,6 @@
     <mti parent="back_husky_bridge" x="0" y="0" z="0.0" rx="0" ry="0" rz="0" />
     <!-- CAMERA macros -->
-    <pointgrey_flea3 prefix="left" parent="front_husky_bridge" base_offset="-0.13" camera_offset="-0.05" camera_r="0" camera_p="0" camera_y="0" />
-    <pointgrey_flea3 prefix="right" parent="front_husky_bridge" base_offset="0.13" camera_offset="0.05" camera_r="0" camera_p="0" camera_y="0" />
+    <pointgrey_flea3 prefix="right" parent="front_husky_bridge" base_offset="-0.13" camera_offset="-0.05" camera_r="0" camera_p="0" camera_y="0" />
+    <pointgrey_flea3 prefix="left" parent="front_husky_bridge" base_offset="0.13" camera_offset="0.05" camera_r="0" camera_p="0" camera_y="0" />
     <!-- PTU-D46 macro -->
     <ptu_d46 parent="front_husky_bridge" x="0" y="-0.025" z="0" rx="0" ry="0" rz="1.5708" />
