Commit message: Changed the Gazebo GPS plugin.

File: urdf/fsr_husky_parts/gps_antenna.urdf.xacro (robot description, xacro)
@@ -63,5 +63,5 @@
     			</collision>
   		</link>
-		<joint name="gps_anetnna_joint" type="fixed">
+		<joint name="gps_antenna_joint" type="fixed">
 			<parent link="${parent}"/>
 			<child link="gps_antenna"/>
@@ -76,7 +76,9 @@
 			  <updateRate>4.0</updateRate>
 			  <bodyName>gps_antenna</bodyName>
+			  <frameId>gps_antenna</frameId>
 			  <topicName>/gps/fix</topicName>
 			  <velocityTopicName>/gps/fix_velocity</velocityTopicName>
-			  <drift>1.0 1.0 1.0</drift>
+			  <offset>0 0 0</offset>
+			  <drift>0.001 0.001 0.001</drift>
 			  <gaussianNoise>0.01 0.01 0.01</gaussianNoise>
 			  <velocityDrift>0 0 0</velocityDrift>
