Commit message: Major update, HRATC2014 ROS packages merging.

File: urdf/arm/fsr_husky_arm.urdf.xacro (robot description, xacro)
@@ -51,5 +51,5 @@
       <geometry>
         <mesh
-          filename="package://hratc2014_simulator/models/arm/base_arm_link.STL" />
+          filename="package://hratc2014_framework/models/arm/base_arm_link.STL" />
       </geometry>
       <material
@@ -65,5 +65,5 @@
       <geometry>
         <mesh
-          filename="package://hratc2014_simulator/models/arm/base_arm_link.STL" />
+          filename="package://hratc2014_framework/models/arm/base_arm_link.STL" />
       </geometry>
     </collision>
@@ -100,5 +100,5 @@
       <geometry>
         <mesh
-          filename="package://hratc2014_simulator/models/arm/arm_axel.STL" />
+          filename="package://hratc2014_framework/models/arm/arm_axel.STL" />
       </geometry>
       <material
@@ -114,5 +114,5 @@
       <geometry>
         <mesh
-          filename="package://hratc2014_simulator/models/arm/arm_axel.STL" />
+          filename="package://hratc2014_framework/models/arm/arm_axel.STL" />
       </geometry>
     </collision>
@@ -162,5 +162,5 @@
       <geometry>
         <mesh
-          filename="package://hratc2014_simulator/models/arm/upper_arm.STL" />
+          filename="package://hratc2014_framework/models/arm/upper_arm.STL" />
       </geometry>
       <material
@@ -176,5 +176,5 @@
       <geometry>
         <mesh
-          filename="package://hratc2014_simulator/models/arm/upper_arm.STL" />
+          filename="package://hratc2014_framework/models/arm/upper_arm.STL" />
       </geometry>
     </collision>
@@ -224,5 +224,5 @@
       <geometry>
         <mesh
-          filename="package://hratc2014_simulator/models/arm/metal_detector_arm.STL" />
+          filename="package://hratc2014_framework/models/arm/metal_detector_arm.STL" />
       </geometry>
       <material
@@ -238,5 +238,5 @@
       <geometry>
         <mesh
-          filename="package://hratc2014_simulator/models/arm/metal_detector_arm.STL" />
+          filename="package://hratc2014_framework/models/arm/metal_detector_arm.STL" />
       </geometry>
     </collision>
@@ -289,5 +289,5 @@
       <geometry>
         <mesh
-          filename="package://hratc2014_simulator/models/arm/metal_detector_antenna.STL" />
+          filename="package://hratc2014_framework/models/arm/metal_detector_antenna.STL" />
       </geometry>
       <material
@@ -303,5 +303,5 @@
       <geometry>
         <mesh
-          filename="package://hratc2014_simulator/models/arm/metal_detector_antenna.STL" />
+          filename="package://hratc2014_framework/models/arm/metal_detector_antenna.STL" />
       </geometry>
     </collision>
@@ -333,5 +333,5 @@
   </link>
   <joint name="left_coil_joint" type="fixed">
-      <origin xyz="0 0 15" rpy="0 0 0" />
+      <origin xyz="0 0.18 0" rpy="0 0 0" />
       <parent link="metal_detector_antenna"/>
       <child link="left_coil" />
@@ -352,5 +352,5 @@
   <link name="right_coil">
       <visual>
-          <origin xyz="0 0 -15" rpy="0 0 0" />
+          <origin xyz="0 0 0" rpy="0 0 0" />
           <geometry>
               <box size="0.001 0.001 0.001" />
@@ -359,5 +359,5 @@
   </link>
   <joint name="right_coil_joint" type="fixed">
-      <origin xyz="0 0 15" rpy="0 0 0" />
+      <origin xyz="0 -0.18 0" rpy="0 0 0" />
       <parent link="metal_detector_antenna"/>
       <child link="right_coil" />
@@ -385,5 +385,5 @@
       <geometry>
         <mesh
-          filename="package://hratc2014_simulator/models/arm/lower_arm.STL" />
+          filename="package://hratc2014_framework/models/arm/lower_arm.STL" />
       </geometry>
       <material
@@ -399,5 +399,5 @@
       <geometry>
         <mesh
-          filename="package://hratc2014_simulator/models/arm/lower_arm.STL" />
+          filename="package://hratc2014_framework/models/arm/lower_arm.STL" />
       </geometry>
     </collision>

File: urdf/fsr_husky_parts/alfa_tube2h.urdf.xacro (robot description, xacro)
@@ -29,5 +29,5 @@
 	xmlns:xacro="http://ros.org/wiki/xacro" name="alfa_tube2h">
 	<!-- Alfa Tube 2H-->
-	<xacro:include filename="$(find hratc2014_simulator)/urdf/fsr_husky_parts/common.xacro" />
+	<xacro:include filename="$(find hratc2014_framework)/urdf/fsr_husky_parts/common.xacro" />
 	<xacro:property name="alfa_length" value="0.132" />
 	<xacro:property name="alfa_radius" value="0.019" />

File: urdf/fsr_husky_parts/gps_antenna.urdf.xacro (robot description, xacro)
@@ -29,5 +29,5 @@
 	xmlns:xacro="http://ros.org/wiki/xacro" name="gps_antenna">
 	<!-- GPS Antenna -->
-	<xacro:include filename="$(find hratc2014_simulator)/urdf/fsr_husky_parts/common.xacro" />
+	<xacro:include filename="$(find hratc2014_framework)/urdf/fsr_husky_parts/common.xacro" />
 	<xacro:property name="alfa_length" value="0.132" />
 	<xacro:property name="alfa_radius" value="0.019" />
@@ -50,5 +50,5 @@
       				<origin xyz="-0.035 0 0" rpy="1.5708 0 0" />
       				<geometry>
-					<mesh filename="package://hratc2014_simulator/models/fsr_husky_parts/gps_antenna.stl" />
+					<mesh filename="package://hratc2014_framework/models/fsr_husky_parts/gps_antenna.stl" />
       				</geometry>
       				<material name="White">
@@ -59,5 +59,5 @@
       				<origin xyz="-0.035 0 0" rpy="1.5708 0 0" />
       				<geometry>
-					<mesh filename="package://hratc2014_simulator/models/fsr_husky_parts/gps_antenna.stl" />
+					<mesh filename="package://hratc2014_framework/models/fsr_husky_parts/gps_antenna.stl" />
      			 	</geometry>
     			</collision>

File: urdf/fsr_husky_parts/husky_bridge.urdf.xacro (robot description, xacro)
@@ -46,5 +46,5 @@
       				<origin xyz="-0.12511 0 ${-bridge_height}" rpy="1.5708 0 1.5708" />
       				<geometry>
-					<mesh filename="package://hratc2014_simulator/models/fsr_husky_parts/bridge.stl" />
+					<mesh filename="package://hratc2014_framework/models/fsr_husky_parts/bridge.stl" />
       				</geometry>
       				<material name="Gray" />
@@ -53,5 +53,5 @@
       				<origin xyz="-0.12511 0 ${-bridge_height}" rpy="1.5708 0 1.5708" />
       				<geometry>
-					<mesh filename="package://hratc2014_simulator/models/fsr_husky_parts/bridge.stl" />
+					<mesh filename="package://hratc2014_framework/models/fsr_husky_parts/bridge.stl" />
       				</geometry>
     			</collision>

File: urdf/fsr_husky_parts/mti.urdf.xacro (robot description, xacro)
@@ -28,5 +28,5 @@
 	xmlns:interface="http://playerstage.sourceforge.net/gazebo/xmlschema/#interface"
 	xmlns:xacro="http://ros.org/wiki/xacro" name="mti">
-	<xacro:include filename="$(find hratc2014_simulator)/urdf/fsr_husky_parts/common.xacro" />
+	<xacro:include filename="$(find hratc2014_framework)/urdf/fsr_husky_parts/common.xacro" />
 	<xacro:property name="mti_length" value="0.057" />
 	<xacro:property name="mti_width" value="0.042" />

File: urdf/fsr_husky_parts/pointgrey_flea3.urdf.xacro (robot description, xacro)
@@ -29,5 +29,5 @@
 	xmlns:xacro="http://ros.org/wiki/xacro" name="pointgrey_flea3">
 	<!-- PointGrey Flea 3 -->
-	<xacro:include filename="$(find hratc2014_simulator)/urdf/fsr_husky_parts/common.xacro" />
+	<xacro:include filename="$(find hratc2014_framework)/urdf/fsr_husky_parts/common.xacro" />
 	<xacro:property name="base_x" value="0.040" />
 	<xacro:property name="base_y" value="0.150" />

File: urdf/fsr_husky_parts/ptu_d46.urdf.xacro (robot description, xacro)
@@ -45,5 +45,5 @@
       				<origin xyz="0 0 0" rpy="0 0 0" />
       				<geometry>
-					<mesh filename="package://hratc2014_simulator/models/fsr_husky_parts/ptu_d46_base_link.stl" />
+					<mesh filename="package://hratc2014_framework/models/fsr_husky_parts/ptu_d46_base_link.stl" />
      	 			</geometry>
       				<material name="DarkGray" />
@@ -52,5 +52,5 @@
       				<origin xyz="0 0 0" rpy="0 0 0" />
       				<geometry>
-					<mesh filename="package://hratc2014_simulator/models/fsr_husky_parts/ptu_d46_base_link.stl" />
+					<mesh filename="package://hratc2014_framework/models/fsr_husky_parts/ptu_d46_base_link.stl" />
       				</geometry>
     			</collision>
@@ -80,5 +80,5 @@
       				<origin xyz="0 0 0" rpy="0 0 0" />
       				<geometry>
-					<mesh filename="package://hratc2014_simulator/models/fsr_husky_parts/ptu_d46_pan_link.stl" />
+					<mesh filename="package://hratc2014_framework/models/fsr_husky_parts/ptu_d46_pan_link.stl" />
       				</geometry>
       				<material name="DarkGray" />
@@ -87,5 +87,5 @@
       				<origin xyz="0 0 0" rpy="0 0 0" />
       				<geometry>
-					<mesh filename="package://hratc2014_simulator/models/fsr_husky_parts/ptu_d46_pan_link.stl" />
+					<mesh filename="package://hratc2014_framework/models/fsr_husky_parts/ptu_d46_pan_link.stl" />
       				</geometry>
     			</collision>
@@ -118,5 +118,5 @@
       				<origin xyz="0 0 0" rpy="0 0 0" />
       				<geometry>
-					<mesh filename="package://hratc2014_simulator/models/fsr_husky_parts/ptu_d46_tilt_link.stl" />
+					<mesh filename="package://hratc2014_framework/models/fsr_husky_parts/ptu_d46_tilt_link.stl" />
       				</geometry>
       				<material name="DarkGray" />
@@ -125,5 +125,5 @@
       				<origin xyz="0 0 0" rpy="0 0 0" />
       				<geometry>
-					<mesh filename="package://hratc2014_simulator/models/fsr_husky_parts/ptu_d46_tilt_link.stl" />
+					<mesh filename="package://hratc2014_framework/models/fsr_husky_parts/ptu_d46_tilt_link.stl" />
       				</geometry>
     			</collision>

File: urdf/fsr_husky_parts/sick_lms100.urdf.xacro (robot description, xacro)
@@ -29,5 +29,5 @@
 	xmlns:xacro="http://ros.org/wiki/xacro" name="sick_lms100">
 	<!-- SICK LMS100-->
-	<xacro:include filename="$(find hratc2014_simulator)/urdf/fsr_husky_parts/common.xacro" />
+	<xacro:include filename="$(find hratc2014_framework)/urdf/fsr_husky_parts/common.xacro" />
 	<xacro:property name="laser_x" value="0.105" />
 	<xacro:property name="laser_y" value="0.102" />
@@ -40,5 +40,5 @@
 				<origin xyz="0 0 0" rpy="0 0 0" />
 				<geometry>
-					<mesh filename="package://hratc2014_simulator/models/fsr_husky_parts/sick_lms100.stl" />
+					<mesh filename="package://hratc2014_framework/models/fsr_husky_parts/sick_lms100.stl" />
 				</geometry>
 				<material name="DarkGray" />
@@ -46,5 +46,5 @@
     			<collision>
       				<geometry>
-					<mesh filename="package://hratc2014_simulator/models/fsr_husky_parts/sick_lms100.stl" />
+					<mesh filename="package://hratc2014_framework/models/fsr_husky_parts/sick_lms100.stl" />
         				<!-- <box size="${laser_x} ${laser_y} ${laser_z}" /> -->
       				</geometry>

File: urdf/husky.urdf.xacro (robot description, xacro)
@@ -42,15 +42,15 @@
     xmlns:xacro="http://ros.org/wiki/xacro" name="husky">
     <!-- Included URDF/XACRO Files -->
-    <xacro:include filename="$(find hratc2014_simulator)/urdf/husky_parts/materials.urdf.xacro" />
-    <xacro:include filename="$(find hratc2014_simulator)/urdf/husky_parts/wheel.urdf.xacro" />
-    <xacro:include filename="$(find hratc2014_simulator)/urdf/husky_parts/parts.urdf.xacro" />
-    <xacro:include filename="$(find hratc2014_simulator)/urdf/fsr_husky_parts/husky_bridge.urdf.xacro" />
-    <xacro:include filename="$(find hratc2014_simulator)/urdf/fsr_husky_parts/sick_lms100.urdf.xacro" />
-    <xacro:include filename="$(find hratc2014_simulator)/urdf/fsr_husky_parts/alfa_tube2h.urdf.xacro" />
-    <xacro:include filename="$(find hratc2014_simulator)/urdf/fsr_husky_parts/pointgrey_flea3.urdf.xacro" />
-    <xacro:include filename="$(find hratc2014_simulator)/urdf/fsr_husky_parts/gps_antenna.urdf.xacro" />
-    <xacro:include filename="$(find hratc2014_simulator)/urdf/fsr_husky_parts/ptu_d46.urdf.xacro" />
-    <xacro:include filename="$(find hratc2014_simulator)/urdf/fsr_husky_parts/mti.urdf.xacro" />
-    <xacro:include filename="$(find hratc2014_simulator)/urdf/arm/fsr_husky_arm.urdf.xacro" />
+    <xacro:include filename="$(find hratc2014_framework)/urdf/husky_parts/materials.urdf.xacro" />
+    <xacro:include filename="$(find hratc2014_framework)/urdf/husky_parts/wheel.urdf.xacro" />
+    <xacro:include filename="$(find hratc2014_framework)/urdf/husky_parts/parts.urdf.xacro" />
+    <xacro:include filename="$(find hratc2014_framework)/urdf/fsr_husky_parts/husky_bridge.urdf.xacro" />
+    <xacro:include filename="$(find hratc2014_framework)/urdf/fsr_husky_parts/sick_lms100.urdf.xacro" />
+    <xacro:include filename="$(find hratc2014_framework)/urdf/fsr_husky_parts/alfa_tube2h.urdf.xacro" />
+    <xacro:include filename="$(find hratc2014_framework)/urdf/fsr_husky_parts/pointgrey_flea3.urdf.xacro" />
+    <xacro:include filename="$(find hratc2014_framework)/urdf/fsr_husky_parts/gps_antenna.urdf.xacro" />
+    <xacro:include filename="$(find hratc2014_framework)/urdf/fsr_husky_parts/ptu_d46.urdf.xacro" />
+    <xacro:include filename="$(find hratc2014_framework)/urdf/fsr_husky_parts/mti.urdf.xacro" />
+    <xacro:include filename="$(find hratc2014_framework)/urdf/arm/fsr_husky_arm.urdf.xacro" />
     <!-- PROPERTY LIST -->
     <!--All units in m-kg-s-radians unit system -->
@@ -113,5 +113,5 @@
             <origin xyz="0 0 0" rpy="0 0 0" />
             <geometry>
-		<mesh filename="package://hratc2014_simulator/models/husky_parts/base_link.stl" />
+		<mesh filename="package://hratc2014_framework/models/husky_parts/base_link.stl" />
             </geometry>
             <material name="Black" />

File: urdf/husky_parts/parts.urdf.xacro (robot description, xacro)
@@ -56,5 +56,5 @@
 				<origin xyz="0 0 0" rpy="0 0 0" />
 				<geometry>
-					<mesh filename="package://hratc2014_simulator/models/husky_parts/${mesh}.stl" />
+					<mesh filename="package://hratc2014_framework/models/husky_parts/${mesh}.stl" />
 				</geometry>
 				<material name="${colour}" />

File: urdf/husky_parts/wheel.urdf.xacro (robot description, xacro)
@@ -58,5 +58,5 @@
 				<origin xyz="0 0 0" rpy="${flipY*M_PI} 0 0" />
 				<geometry>
-					<mesh filename="package://hratc2014_simulator/models/husky_parts/wheel.stl" />
+					<mesh filename="package://hratc2014_framework/models/husky_parts/wheel.stl" />
 				</geometry>
 				<material name="DarkGray" />

Commit message: Adiciona movimento do braço do sensor no gazebo ao framework

File: urdf/arm/fsr_husky_arm.urdf.xacro (robot description, xacro)
@@ -333,5 +333,5 @@
   </link>
   <joint name="left_coil_joint" type="fixed">
-      <origin xyz="0 0.18 0" rpy="0 0 0" />
+      <origin xyz="0.18 0 0" rpy="0 0 0" />
       <parent link="metal_detector_antenna"/>
       <child link="left_coil" />
@@ -359,5 +359,5 @@
   </link>
   <joint name="right_coil_joint" type="fixed">
-      <origin xyz="0 -0.18 0" rpy="0 0 0" />
+      <origin xyz="-0.18 0 0" rpy="0 0 0" />
       <parent link="metal_detector_antenna"/>
       <child link="right_coil" />

Commit message: Major update to the controllers interface.

File: urdf/arm/fsr_husky_arm.urdf.xacro (robot description, xacro)
@@ -459,9 +459,9 @@
     </actuator>
   </transmission>
-  <gazebo>
+  <!--<gazebo>
     <plugin name="gazebo_ros_control" filename="libgazebo_ros_control.so">
       <robotNamespace>/arm</robotNamespace>
     </plugin>
-  </gazebo>
+  </gazebo>-->
 </xacro:macro>
 </robot>

File: urdf/fsr_husky_parts/ptu_d46.urdf.xacro (robot description, xacro)
@@ -134,5 +134,5 @@
     		</gazebo>
 		<joint name="ptu_d46_tilt_joint" type="revolute">
-    			<origin xyz="0 0 0.0455" rpy="1.5708 0 0" />
+    			<origin xyz="0 0 0.0455" rpy="1.3 0 0" />
     			<parent link="ptu_d46_pan_link" />
     			<child link="ptu_d46_tilt_link" />
@@ -157,9 +157,9 @@
 		  </actuator>
 		</transmission>
-		<gazebo>
+		<!--<gazebo>
 		  <plugin name="gazebo_ros_control" filename="libgazebo_ros_control.so">
 		    <robotNamespace>/ptu_d46</robotNamespace>
 		  </plugin>
-		</gazebo>
+		</gazebo>-->
 	</xacro:macro>
 </robot>

File: urdf/fsr_husky_parts/sick_lms100.urdf.xacro (robot description, xacro)
@@ -58,8 +58,8 @@
 		<gazebo reference="sick_lms100">
 			<material>Gazebo/Grey</material>
-			<turnGravityOff>true</turnGravityOff>
-    			<sensor type="gpu_ray" name="sick_lms100">
+			<turnGravityOff>false</turnGravityOff>
+    			<sensor type="ray" name="sick_lms100">
       				<pose>0 0 0 0 0 0</pose>
-      				<visualize>false</visualize>
+      				<visualize>true</visualize>
      	 			<update_rate>40</update_rate>
       				<ray>
@@ -83,5 +83,5 @@
         				</noise>
       				</ray>
-      				<plugin name="gazebo_ros_laser" filename="libgazebo_ros_gpu_laser.so">
+      				<plugin name="gazebo_ros_laser" filename="libgazebo_ros_laser.so">
         				<topicName>scan</topicName>
         				<frameName>sick_lms100</frameName>

File: urdf/husky.urdf.xacro (robot description, xacro)
@@ -197,3 +197,8 @@
     <!-- FSR Husky De-mining Arm -->
     <fsr_husky_arm parent="base_link" x="0.120" y="-0.15" z="${base_z_size}" rx="0" ry="0" rz="0" />
+    <gazebo>
+      <plugin name="gazebo_ros_control" filename="libgazebo_ros_control.so">
+	<!--<robotNamespace>/husky</robotNamespace>-->
+      </plugin>
+    </gazebo>
 </robot>

Commit message: Major update to bring the arm simulation closer to the real Husky.

File: urdf/arm/fsr_husky_arm.urdf.xacro (robot description, xacro)
@@ -137,5 +137,5 @@
       lower="-1.5708"
       upper="1.5708"
-      effort="100"
+      effort="15"
       velocity="0.5" />
   </joint>
@@ -199,5 +199,5 @@
       lower="-0.5"
       upper="0.25"
-      effort="20"
+      effort="15"
       velocity="0.5" />
   </joint>
@@ -264,5 +264,5 @@
       lower="-0.25"
       upper="0.5"
-      effort="20"
+      effort="15"
       velocity="0.5" />
   </joint>
@@ -424,27 +424,11 @@
       lower="-0.5"
       upper="0.25"
-      effort="20"
+      effort="15"
       velocity="0.5" />
   </joint>
-  <transmission name="upper_lift">
+  <transmission name="lift">
     <type>transmission_interface/SimpleTransmission</type>
     <joint name="upper_arm_joint"/>
-    <actuator name="upper_lift_motor">
-      <hardwareInterface>EffortJointInterface</hardwareInterface>
-      <mechanicalReduction>1</mechanicalReduction>
-    </actuator>
-  </transmission>
-  <transmission name="lower_lift">
-    <type>transmission_interface/SimpleTransmission</type>
-    <joint name="lower_arm_joint"/>
-    <actuator name="lower_lift_motor">
-      <hardwareInterface>EffortJointInterface</hardwareInterface>
-      <mechanicalReduction>1</mechanicalReduction>
-    </actuator>
-  </transmission>
-  <transmission name="mirror_lift">
-    <type>transmission_interface/SimpleTransmission</type>
-    <joint name="metal_detector_arm_joint"/>
-    <actuator name="mirror_lift_motor">
+    <actuator name="lift_motor">
       <hardwareInterface>EffortJointInterface</hardwareInterface>
       <mechanicalReduction>1</mechanicalReduction>
@@ -459,9 +443,18 @@
     </actuator>
   </transmission>
-  <!--<gazebo>
-    <plugin name="gazebo_ros_control" filename="libgazebo_ros_control.so">
-      <robotNamespace>/arm</robotNamespace>
-    </plugin>
-  </gazebo>-->
+  <gazebo>
+	<plugin name="mimic_plugin1" filename="libgazebo_mimic_plugin.so">
+            <joint>upper_arm_joint</joint>
+            <mimicJoint>lower_arm_joint</mimicJoint>
+            <multiplier>1.0</multiplier>
+        </plugin>
+  </gazebo>
+  <gazebo>
+	<plugin name="mimic_plugin2" filename="libgazebo_mimic_plugin.so">
+            <joint>upper_arm_joint</joint>
+            <mimicJoint>metal_detector_arm_joint</mimicJoint>
+            <multiplier>-1.0</multiplier>
+        </plugin>
+  </gazebo>
 </xacro:macro>
 </robot>

Commit message: Fixing a broken tf tree on the arm.

File: urdf/arm/fsr_husky_arm.urdf.xacro (robot description, xacro)
@@ -435,4 +435,20 @@
     </actuator>
   </transmission>
+  <transmission name="mimic_lift">
+    <type>transmission_interface/SimpleTransmission</type>
+    <joint name="lower_arm_joint"/>
+    <actuator name="mimic_lift_motor">
+      <hardwareInterface>EffortJointInterface</hardwareInterface>
+      <mechanicalReduction>1</mechanicalReduction>
+    </actuator>
+  </transmission>
+  <transmission name="mirror_lift">
+    <type>transmission_interface/SimpleTransmission</type>
+    <joint name="metal_detector_arm_joint"/>
+    <actuator name="mirror_lift_motor">
+      <hardwareInterface>EffortJointInterface</hardwareInterface>
+      <mechanicalReduction>1</mechanicalReduction>
+    </actuator>
+  </transmission>
   <transmission name="sweep">
     <type>transmission_interface/SimpleTransmission</type>
