Commit message: Adapting package names

File: urdf/arm/fsr_husky_arm.urdf.xacro (robot description, xacro)
@@ -51,5 +51,5 @@
       <geometry>
         <mesh
-          filename="package://hratc2014_framework/models/arm/base_arm_link.STL" />
+          filename="package://hratc2015_framework/models/arm/base_arm_link.STL" />
       </geometry>
       <material
@@ -65,5 +65,5 @@
       <geometry>
         <mesh
-          filename="package://hratc2014_framework/models/arm/base_arm_link.STL" />
+          filename="package://hratc2015_framework/models/arm/base_arm_link.STL" />
       </geometry>
     </collision>
@@ -100,5 +100,5 @@
       <geometry>
         <mesh
-          filename="package://hratc2014_framework/models/arm/arm_axel.STL" />
+          filename="package://hratc2015_framework/models/arm/arm_axel.STL" />
       </geometry>
       <material
@@ -114,5 +114,5 @@
       <geometry>
         <mesh
-          filename="package://hratc2014_framework/models/arm/arm_axel.STL" />
+          filename="package://hratc2015_framework/models/arm/arm_axel.STL" />
       </geometry>
     </collision>
@@ -162,5 +162,5 @@
       <geometry>
         <mesh
-          filename="package://hratc2014_framework/models/arm/upper_arm.STL" />
+          filename="package://hratc2015_framework/models/arm/upper_arm.STL" />
       </geometry>
       <material
@@ -176,5 +176,5 @@
       <geometry>
         <mesh
-          filename="package://hratc2014_framework/models/arm/upper_arm.STL" />
+          filename="package://hratc2015_framework/models/arm/upper_arm.STL" />
       </geometry>
     </collision>
@@ -224,5 +224,5 @@
       <geometry>
         <mesh
-          filename="package://hratc2014_framework/models/arm/metal_detector_arm.STL" />
+          filename="package://hratc2015_framework/models/arm/metal_detector_arm.STL" />
       </geometry>
       <material
@@ -238,5 +238,5 @@
       <geometry>
         <mesh
-          filename="package://hratc2014_framework/models/arm/metal_detector_arm.STL" />
+          filename="package://hratc2015_framework/models/arm/metal_detector_arm.STL" />
       </geometry>
     </collision>
@@ -289,5 +289,5 @@
       <geometry>
         <mesh
-          filename="package://hratc2014_framework/models/arm/metal_detector_antenna.STL" />
+          filename="package://hratc2015_framework/models/arm/metal_detector_antenna.STL" />
       </geometry>
       <material
@@ -303,5 +303,5 @@
       <geometry>
         <mesh
-          filename="package://hratc2014_framework/models/arm/metal_detector_antenna.STL" />
+          filename="package://hratc2015_framework/models/arm/metal_detector_antenna.STL" />
       </geometry>
     </collision>
@@ -385,5 +385,5 @@
       <geometry>
         <mesh
-          filename="package://hratc2014_framework/models/arm/lower_arm.STL" />
+          filename="package://hratc2015_framework/models/arm/lower_arm.STL" />
       </geometry>
       <material
@@ -399,5 +399,5 @@
       <geometry>
         <mesh
-          filename="package://hratc2014_framework/models/arm/lower_arm.STL" />
+          filename="package://hratc2015_framework/models/arm/lower_arm.STL" />
       </geometry>
     </collision>

File: urdf/fsr_husky_parts/alfa_tube2h.urdf.xacro (robot description, xacro)
@@ -29,5 +29,5 @@
 	xmlns:xacro="http://ros.org/wiki/xacro" name="alfa_tube2h">
 	<!-- Alfa Tube 2H-->
-	<xacro:include filename="$(find hratc2014_framework)/urdf/fsr_husky_parts/common.xacro" />
+	<xacro:include filename="$(find hratc2015_framework)/urdf/fsr_husky_parts/common.xacro" />
 	<xacro:property name="alfa_length" value="0.132" />
 	<xacro:property name="alfa_radius" value="0.019" />

File: urdf/fsr_husky_parts/gps_antenna.urdf.xacro (robot description, xacro)
@@ -29,5 +29,5 @@
 	xmlns:xacro="http://ros.org/wiki/xacro" name="gps_antenna">
 	<!-- GPS Antenna -->
-	<xacro:include filename="$(find hratc2014_framework)/urdf/fsr_husky_parts/common.xacro" />
+	<xacro:include filename="$(find hratc2015_framework)/urdf/fsr_husky_parts/common.xacro" />
 	<xacro:property name="alfa_length" value="0.132" />
 	<xacro:property name="alfa_radius" value="0.019" />
@@ -50,5 +50,5 @@
       				<origin xyz="-0.035 0 0" rpy="1.5708 0 0" />
       				<geometry>
-					<mesh filename="package://hratc2014_framework/models/fsr_husky_parts/gps_antenna.stl" />
+					<mesh filename="package://hratc2015_framework/models/fsr_husky_parts/gps_antenna.stl" />
       				</geometry>
       				<material name="White">
@@ -59,5 +59,5 @@
       				<origin xyz="-0.035 0 0" rpy="1.5708 0 0" />
       				<geometry>
-					<mesh filename="package://hratc2014_framework/models/fsr_husky_parts/gps_antenna.stl" />
+					<mesh filename="package://hratc2015_framework/models/fsr_husky_parts/gps_antenna.stl" />
      			 	</geometry>
     			</collision>

File: urdf/fsr_husky_parts/husky_bridge.urdf.xacro (robot description, xacro)
@@ -46,5 +46,5 @@
       				<origin xyz="-0.12511 0 ${-bridge_height}" rpy="1.5708 0 1.5708" />
       				<geometry>
-					<mesh filename="package://hratc2014_framework/models/fsr_husky_parts/bridge.stl" />
+					<mesh filename="package://hratc2015_framework/models/fsr_husky_parts/bridge.stl" />
       				</geometry>
       				<material name="Gray" />
@@ -53,5 +53,5 @@
       				<origin xyz="-0.12511 0 ${-bridge_height}" rpy="1.5708 0 1.5708" />
       				<geometry>
-					<mesh filename="package://hratc2014_framework/models/fsr_husky_parts/bridge.stl" />
+					<mesh filename="package://hratc2015_framework/models/fsr_husky_parts/bridge.stl" />
       				</geometry>
     			</collision>

File: urdf/fsr_husky_parts/mti.urdf.xacro (robot description, xacro)
@@ -28,5 +28,5 @@
 	xmlns:interface="http://playerstage.sourceforge.net/gazebo/xmlschema/#interface"
 	xmlns:xacro="http://ros.org/wiki/xacro" name="mti">
-	<xacro:include filename="$(find hratc2014_framework)/urdf/fsr_husky_parts/common.xacro" />
+	<xacro:include filename="$(find hratc2015_framework)/urdf/fsr_husky_parts/common.xacro" />
 	<xacro:property name="mti_length" value="0.057" />
 	<xacro:property name="mti_width" value="0.042" />

File: urdf/fsr_husky_parts/pointgrey_flea3.urdf.xacro (robot description, xacro)
@@ -29,5 +29,5 @@
 	xmlns:xacro="http://ros.org/wiki/xacro" name="pointgrey_flea3">
 	<!-- PointGrey Flea 3 -->
-	<xacro:include filename="$(find hratc2014_framework)/urdf/fsr_husky_parts/common.xacro" />
+	<xacro:include filename="$(find hratc2015_framework)/urdf/fsr_husky_parts/common.xacro" />
 	<xacro:property name="base_x" value="0.040" />
 	<xacro:property name="base_y" value="0.150" />

File: urdf/fsr_husky_parts/ptu_d46.urdf.xacro (robot description, xacro)
@@ -45,5 +45,5 @@
       				<origin xyz="0 0 0" rpy="0 0 0" />
       				<geometry>
-					<mesh filename="package://hratc2014_framework/models/fsr_husky_parts/ptu_d46_base_link.stl" />
+					<mesh filename="package://hratc2015_framework/models/fsr_husky_parts/ptu_d46_base_link.stl" />
      	 			</geometry>
       				<material name="DarkGray" />
@@ -52,5 +52,5 @@
       				<origin xyz="0 0 0" rpy="0 0 0" />
       				<geometry>
-					<mesh filename="package://hratc2014_framework/models/fsr_husky_parts/ptu_d46_base_link.stl" />
+					<mesh filename="package://hratc2015_framework/models/fsr_husky_parts/ptu_d46_base_link.stl" />
       				</geometry>
     			</collision>
@@ -80,5 +80,5 @@
       				<origin xyz="0 0 0" rpy="0 0 0" />
       				<geometry>
-					<mesh filename="package://hratc2014_framework/models/fsr_husky_parts/ptu_d46_pan_link.stl" />
+					<mesh filename="package://hratc2015_framework/models/fsr_husky_parts/ptu_d46_pan_link.stl" />
       				</geometry>
       				<material name="DarkGray" />
@@ -87,5 +87,5 @@
       				<origin xyz="0 0 0" rpy="0 0 0" />
       				<geometry>
-					<mesh filename="package://hratc2014_framework/models/fsr_husky_parts/ptu_d46_pan_link.stl" />
+					<mesh filename="package://hratc2015_framework/models/fsr_husky_parts/ptu_d46_pan_link.stl" />
       				</geometry>
     			</collision>
@@ -118,5 +118,5 @@
       				<origin xyz="0 0 0" rpy="0 0 0" />
       				<geometry>
-					<mesh filename="package://hratc2014_framework/models/fsr_husky_parts/ptu_d46_tilt_link.stl" />
+					<mesh filename="package://hratc2015_framework/models/fsr_husky_parts/ptu_d46_tilt_link.stl" />
       				</geometry>
       				<material name="DarkGray" />
@@ -125,5 +125,5 @@
       				<origin xyz="0 0 0" rpy="0 0 0" />
       				<geometry>
-					<mesh filename="package://hratc2014_framework/models/fsr_husky_parts/ptu_d46_tilt_link.stl" />
+					<mesh filename="package://hratc2015_framework/models/fsr_husky_parts/ptu_d46_tilt_link.stl" />
       				</geometry>
     			</collision>

File: urdf/fsr_husky_parts/sick_lms100.urdf.xacro (robot description, xacro)
@@ -29,5 +29,5 @@
 	xmlns:xacro="http://ros.org/wiki/xacro" name="sick_lms100">
 	<!-- SICK LMS100-->
-	<xacro:include filename="$(find hratc2014_framework)/urdf/fsr_husky_parts/common.xacro" />
+	<xacro:include filename="$(find hratc2015_framework)/urdf/fsr_husky_parts/common.xacro" />
 	<xacro:property name="laser_x" value="0.105" />
 	<xacro:property name="laser_y" value="0.102" />
@@ -40,5 +40,5 @@
 				<origin xyz="0 0 0" rpy="0 0 0" />
 				<geometry>
-					<mesh filename="package://hratc2014_framework/models/fsr_husky_parts/sick_lms100.stl" />
+					<mesh filename="package://hratc2015_framework/models/fsr_husky_parts/sick_lms100.stl" />
 				</geometry>
 				<material name="DarkGray" />
@@ -46,5 +46,5 @@
     			<collision>
       				<geometry>
-					<mesh filename="package://hratc2014_framework/models/fsr_husky_parts/sick_lms100.stl" />
+					<mesh filename="package://hratc2015_framework/models/fsr_husky_parts/sick_lms100.stl" />
         				<!-- <box size="${laser_x} ${laser_y} ${laser_z}" /> -->
       				</geometry>

File: urdf/gps.urdf.xacro (robot description, xacro)
@@ -24,5 +24,5 @@
 (INCLUDING NEGLIGENCE OR OTHERWISE) ARISING IN ANY WAY OUT OF THE USE OF THIS
 SOFTWARE, EVEN IF ADVISED OF THE POSSIBILITY OF SUCH DAMAGE.
-This program contains the description of the HRATC2014 Husky robot based on the original Clearpath
+This program contains the description of the HRATC2015 Husky robot based on the original Clearpath
 Husky A200 file and modified by the ISR University of Coimbra
 -->
@@ -42,5 +42,5 @@
     xmlns:xacro="http://ros.org/wiki/xacro" name="husky">
     <!-- Included URDF/XACRO Files -->
-    <xacro:include filename="$(find hratc2014_framework)/urdf/fsr_husky_parts/gps_antenna.urdf.xacro" />
+    <xacro:include filename="$(find hratc2015_framework)/urdf/fsr_husky_parts/gps_antenna.urdf.xacro" />
     <link name="base_footprint">
         <!--<inertial>
@@ -73,5 +73,5 @@
       				<origin xyz="-0.035 0 0" rpy="1.5708 0 0" />
       				<geometry>
-					<mesh filename="package://hratc2014_framework/models/fsr_husky_parts/gps_antenna.stl" />
+					<mesh filename="package://hratc2015_framework/models/fsr_husky_parts/gps_antenna.stl" />
       				</geometry>
       				<material name="White">
@@ -82,5 +82,5 @@
       				<origin xyz="-0.035 0 0" rpy="1.5708 0 0" />
       				<geometry>
-					<mesh filename="package://hratc2014_framework/models/fsr_husky_parts/gps_antenna.stl" />
+					<mesh filename="package://hratc2015_framework/models/fsr_husky_parts/gps_antenna.stl" />
      			 	</geometry>
     			</collision>

File: urdf/husky.urdf.xacro (robot description, xacro)
@@ -24,5 +24,5 @@
 (INCLUDING NEGLIGENCE OR OTHERWISE) ARISING IN ANY WAY OUT OF THE USE OF THIS
 SOFTWARE, EVEN IF ADVISED OF THE POSSIBILITY OF SUCH DAMAGE.
-This program contains the description of the HRATC2014 Husky robot based on the original Clearpath
+This program contains the description of the HRATC2015 Husky robot based on the original Clearpath
 Husky A200 file and modified by the ISR University of Coimbra
 -->
@@ -42,15 +42,15 @@
     xmlns:xacro="http://ros.org/wiki/xacro" name="husky">
     <!-- Included URDF/XACRO Files -->
-    <xacro:include filename="$(find hratc2014_framework)/urdf/husky_parts/materials.urdf.xacro" />
-    <xacro:include filename="$(find hratc2014_framework)/urdf/husky_parts/wheel.urdf.xacro" />
-    <xacro:include filename="$(find hratc2014_framework)/urdf/husky_parts/parts.urdf.xacro" />
-    <xacro:include filename="$(find hratc2014_framework)/urdf/fsr_husky_parts/husky_bridge.urdf.xacro" />
-    <xacro:include filename="$(find hratc2014_framework)/urdf/fsr_husky_parts/sick_lms100.urdf.xacro" />
-    <xacro:include filename="$(find hratc2014_framework)/urdf/fsr_husky_parts/alfa_tube2h.urdf.xacro" />
-    <xacro:include filename="$(find hratc2014_framework)/urdf/fsr_husky_parts/pointgrey_flea3.urdf.xacro" />
-    <xacro:include filename="$(find hratc2014_framework)/urdf/fsr_husky_parts/gps_antenna.urdf.xacro" />
-    <xacro:include filename="$(find hratc2014_framework)/urdf/fsr_husky_parts/ptu_d46.urdf.xacro" />
-    <xacro:include filename="$(find hratc2014_framework)/urdf/fsr_husky_parts/mti.urdf.xacro" />
-    <xacro:include filename="$(find hratc2014_framework)/urdf/arm/fsr_husky_arm.urdf.xacro" />
+    <xacro:include filename="$(find hratc2015_framework)/urdf/husky_parts/materials.urdf.xacro" />
+    <xacro:include filename="$(find hratc2015_framework)/urdf/husky_parts/wheel.urdf.xacro" />
+    <xacro:include filename="$(find hratc2015_framework)/urdf/husky_parts/parts.urdf.xacro" />
+    <xacro:include filename="$(find hratc2015_framework)/urdf/fsr_husky_parts/husky_bridge.urdf.xacro" />
+    <xacro:include filename="$(find hratc2015_framework)/urdf/fsr_husky_parts/sick_lms100.urdf.xacro" />
+    <xacro:include filename="$(find hratc2015_framework)/urdf/fsr_husky_parts/alfa_tube2h.urdf.xacro" />
+    <xacro:include filename="$(find hratc2015_framework)/urdf/fsr_husky_parts/pointgrey_flea3.urdf.xacro" />
+    <xacro:include filename="$(find hratc2015_framework)/urdf/fsr_husky_parts/gps_antenna.urdf.xacro" />
+    <xacro:include filename="$(find hratc2015_framework)/urdf/fsr_husky_parts/ptu_d46.urdf.xacro" />
+    <xacro:include filename="$(find hratc2015_framework)/urdf/fsr_husky_parts/mti.urdf.xacro" />
+    <xacro:include filename="$(find hratc2015_framework)/urdf/arm/fsr_husky_arm.urdf.xacro" />
     <!-- PROPERTY LIST -->
     <!--All units in m-kg-s-radians unit system -->
@@ -113,5 +113,5 @@
             <origin xyz="0 0 0" rpy="0 0 0" />
             <geometry>
-		<mesh filename="package://hratc2014_framework/models/husky_parts/base_link.stl" />
+		<mesh filename="package://hratc2015_framework/models/husky_parts/base_link.stl" />
             </geometry>
             <material name="Black" />

File: urdf/husky_parts/parts.urdf.xacro (robot description, xacro)
@@ -56,5 +56,5 @@
 				<origin xyz="0 0 0" rpy="0 0 0" />
 				<geometry>
-					<mesh filename="package://hratc2014_framework/models/husky_parts/${mesh}.stl" />
+					<mesh filename="package://hratc2015_framework/models/husky_parts/${mesh}.stl" />
 				</geometry>
 				<material name="${colour}" />

File: urdf/husky_parts/wheel.urdf.xacro (robot description, xacro)
@@ -58,5 +58,5 @@
 				<origin xyz="0 0 0" rpy="${flipY*M_PI} 0 0" />
 				<geometry>
-					<mesh filename="package://hratc2014_framework/models/husky_parts/wheel.stl" />
+					<mesh filename="package://hratc2015_framework/models/husky_parts/wheel.stl" />
 				</geometry>
 				<material name="DarkGray" />
