Commit message: Update to the URDF model for the new Husky

File: urdf/arm/fsr_husky_arm.urdf.xacro (robot description, xacro)
@@ -33,15 +33,15 @@
     <inertial>
       <origin
-        xyz="0.0748500402726595 0.0136470618219005 -0.0925164110070736"
-        rpy="0 0 0" />
-      <mass
-        value="0.215286927386896" />
-      <inertia
-        ixx="0.00151952875960782"
-        ixy="-5.00239624175035E-05"
-        ixz="-0.000104007201846032"
-        iyy="0.00181155299285244"
-        iyz="0.000216578123822788"
-        izz="0.000582288664758318" />
+        xyz="0.062584 0.18878 0.37271"
+        rpy="0 0 0" />
+      <mass
+        value="0.85803" />
+      <inertia
+        ixx="0.0087778"
+        ixy="-0.00034853"
+        ixz="0.0010654"
+        iyy="0.014921"
+        iyz="-0.0021847"
+        izz="0.01488" />
     </inertial>
     <visual>
@@ -53,9 +53,5 @@
           filename="package://hratc2015_framework/models/arm/base_arm_link.STL" />
       </geometry>
-      <material
-        name="Gray">
-        <color
-          rgba="0.776470588235294 0.756862745098039 0.737254901960784 1" />
-      </material>
+      <material name="Black" />
     </visual>
     <collision>
@@ -70,5 +66,6 @@
   </link>
   <gazebo reference="base_arm_link">
-        <material>Gazebo/Grey</material>
+        <material>Gazebo/Black</material>
+	<selfCollide>false</selfCollide>
         <turnGravityOff>true</turnGravityOff>
     </gazebo>
@@ -82,15 +79,15 @@
     <inertial>
       <origin
-        xyz="-6.71167554128979E-05 0.147555068632442 -5.01352348164508E-07"
-        rpy="0 0 0" />
-      <mass
-        value="0.116752432749066" />
-      <inertia
-        ixx="0.000715149281043979"
-        ixy="7.80945806556874E-07"
-        ixz="6.95759354868419E-10"
-        iyy="8.63256490972112E-06"
-        iyz="-1.92225108206073E-09"
-        izz="0.000715441962309322" />
+        xyz="-0.0045492 0.35516 -0.025701"
+        rpy="0 0 0" />
+      <mass
+        value="0.49315" />
+      <inertia
+        ixx="0.0060272"
+        ixy="-0.00056478"
+        ixz="8.6784E-05"
+        iyy="0.0010748"
+        iyz="-0.00058695"
+        izz="0.0064909" />
     </inertial>
     <visual>
@@ -103,5 +100,5 @@
       </geometry>
       <material
-        name="Gray">
+        name="DarkGray">
         <color
           rgba="0.776470588235294 0.756862745098039 0.737254901960784 1" />
@@ -120,4 +117,5 @@
   <gazebo reference="arm_axel">
         <material>Gazebo/Grey</material>
+        <selfCollide>false</selfCollide>
         <turnGravityOff>true</turnGravityOff>
     </gazebo>
@@ -126,6 +124,6 @@
     type="revolute">
     <origin
-      xyz="0.06 0.152 0"
-      rpy="1.5708 0 0" />
+      xyz="0.12828 -0.4402 0.049088"
+      rpy="1.5708 6.123E-17 1.5708" />
     <parent
       link="base_arm_link" />
@@ -134,9 +132,9 @@
     <axis
       xyz="0 -1 0" />
-    <limit
+	<limit
       lower="-1.5708"
-      upper="1.5708"
-      effort="15"
-      velocity="0.5" />
+      upper="3.14"
+      effort="75"
+      velocity="2" />
   </joint>
   <link
@@ -144,15 +142,15 @@
     <inertial>
       <origin
-        xyz="0.000102539584510564 0.025319004836415 0.373317706752181"
-        rpy="0 0 0" />
-      <mass
-        value="0.310661228623748" />
-      <inertia
-        ixx="0.0301188716585458"
-        ixy="-4.68610675580059E-08"
-        ixz="1.48034298202518E-05"
-        iyy="0.0301182394443099"
-        iyz="-0.000152720615635198"
-        izz="8.7451640283179E-05" />
+        xyz="9.76184988289996E-05 0.0241578589661459 0.355397722899461"
+        rpy="0 0 0" />
+      <mass
+        value="0.326325490126923" />
+      <inertia
+        ixx="0.0322020258970473"
+        ixy="-4.4638355127408E-08"
+        ixz="1.53741858406116E-05"
+        iyy="0.032199356997134"
+        iyz="-0.000144641063316242"
+        izz="9.23314207900664E-05" />
     </inertial>
     <visual>
@@ -182,4 +180,5 @@
   <gazebo reference="upper_arm">
         <material>Gazebo/Grey</material>
+        <selfCollide>false</selfCollide>
         <turnGravityOff>true</turnGravityOff>
     </gazebo>
@@ -188,6 +187,6 @@
     type="revolute">
     <origin
-      xyz="0 0.1459 -0.0096445"
-      rpy="-1.5708 0 -1.5708" />
+      xyz="0 0.44 0.011736"
+      rpy="1.5708 0 -1.5708" />
     <parent
       link="arm_axel" />
@@ -195,10 +194,10 @@
       link="upper_arm" />
     <axis
-      xyz="0 1 0" />
+      xyz="0 -1 0" />
     <limit
-      lower="-0.5"
-      upper="0.25"
-      effort="15"
-      velocity="0.5" />
+      lower="-0.5236"
+      upper="0.5236"
+      effort="35"
+      velocity="2" />
   </joint>
   <link
@@ -206,15 +205,15 @@
     <inertial>
       <origin
-        xyz="0.00200170148149059 -0.0639004587205252 -0.0667324909004516"
-        rpy="0 0 0" />
-      <mass
-	value="0.00001" /><!--value="0.730115545526703" />-->
-      <inertia
-        ixx="0.00564260404067653"
-        ixy="4.21272987506857E-05"
-        ixz="4.78655101148471E-05"
-        iyy="0.00114533989924875"
-        iyz="0.00095063627641457"
-        izz="0.00479397824386875" />
+        xyz="-0.0131202075717661 -0.0723031614133108 -0.0463889610764896"
+        rpy="0 0 0" />
+      <mass
+        value="0.730115578586952" />
+      <inertia
+        ixx="0.00493443507445138"
+        ixy="-0.000620294299504152"
+        ixz="-0.000306843036961987"
+        iyy="0.0014212633147968"
+        iyz="0.00125817384513895"
+        izz="0.00527185766074029" />
     </inertial>
     <visual>
@@ -244,4 +243,5 @@
   <gazebo reference="metal_detector_arm">
         <material>Gazebo/Grey</material>
+        <selfCollide>false</selfCollide>
         <turnGravityOff>true</turnGravityOff>
     </gazebo>
@@ -253,6 +253,6 @@
       multiplier="-1" />
     <origin
-      xyz="0 0 0.8475"
-      rpy="1.5708 -1.5708 0" />
+      xyz="-0.783340615005693 0.189233712627677 0.0344999999999998"
+      rpy="-1.5707963267949 1.140744854051 -1.26098072342103" />
     <parent
       link="upper_arm" />
@@ -260,10 +260,10 @@
       link="metal_detector_arm" />
     <axis
-      xyz="0 0 -1" />
-    <limit
-      lower="-0.25"
-      upper="0.5"
-      effort="15"
-      velocity="0.5" />
+      xyz="0.397068061333986 -0.865669276483222 -0.30488302416088" />
+	<limit
+      lower="-0.5236"
+      upper="0.5236"
+      effort="35"
+      velocity="2" />
   </joint>
   <link
@@ -271,15 +271,15 @@
     <inertial>
       <origin
-        xyz="3.6833E-07 0.011468 -0.12477"
-        rpy="0 0 0" />
-      <mass
-	value="0.00001" /><!--value="12.099" />-->
-      <inertia
-        ixx="0.060468"
-        ixy="-4.3221E-09"
-        ixz="5.3405E-07"
-        iyy="0.27654"
-        iyz="-0.0010461"
-        izz="0.21765" />
+        xyz="0.124781096368378 -0.279414752184092 -0.122957072146209"
+        rpy="0 0 0" />
+      <mass
+        value="12.0992798706323" />
+      <inertia
+        ixx="0.223638341370907"
+        ixy="0.0140547266307369"
+        ixz="0.0258666395393033"
+        iyy="0.250461845552196"
+        iyz="-0.0571594766057374"
+        izz="0.0805524351506661" />
     </inertial>
     <visual>
@@ -309,4 +309,5 @@
   <gazebo reference="metal_detector_antenna">
         <material>Gazebo/Green</material>
+        <selfCollide>false</selfCollide>
         <turnGravityOff>true</turnGravityOff>
     </gazebo>
@@ -315,6 +316,6 @@
     type="fixed">
     <origin
-      xyz="0 -0.33276 0.095344"
-      rpy="0 0 0" />
+      xyz="0 0 0"
+      rpy="0 -2.7756E-17 -1.3878E-17" />
     <parent
       link="metal_detector_arm" />
@@ -367,15 +368,15 @@
     <inertial>
       <origin
-        xyz="-4.03262433168461E-08 0.0238835580685394 0.38020982511275"
-        rpy="0 0 0" />
-      <mass
-        value="0.315289032495142" />
-      <inertia
-        ixx="0.0311225242878348"
-        ixy="-2.44666563034439E-10"
-        ixz="3.98116348654419E-09"
-        iyy="0.0311222097229973"
-        iyz="-0.000155853742938512"
-        izz="8.78358578959995E-05" />
+        xyz="-0.234602780446024 -0.225204746125893 0.0031580399460546"
+        rpy="0 0 0" />
+      <mass
+        value="1.27837430758482" />
+      <inertia
+        ixx="0.0167023392786261"
+        ixy="0.0172620654204666"
+        ixz="0.00171207285568604"
+        iyy="0.0255068597107398"
+        iyz="0.000242235271108958"
+        izz="0.0382877611003989" />
     </inertial>
     <visual>
@@ -405,4 +406,5 @@
   <gazebo reference="lower_arm">
         <material>Gazebo/Grey</material>
+        <selfCollide>false</selfCollide>
         <turnGravityOff>true</turnGravityOff>
     </gazebo>
@@ -413,6 +415,6 @@
       joint="upper_arm_joint" />
     <origin
-      xyz="0 0.0809 -0.011058"
-      rpy="-1.5708 0 -1.5708" />
+      xyz="0 0.375 0"
+      rpy="3.1416 0 0.70689" />
     <parent
       link="arm_axel" />
@@ -420,11 +422,12 @@
       link="lower_arm" />
     <axis
-      xyz="0 1 0" />
+      xyz="0 0 1" />
     <limit
-      lower="-0.5"
-      upper="0.25"
-      effort="15"
-      velocity="0.5" />
-  </joint>
+      lower="-0.5236"
+      upper="0.5236"
+      effort="35"
+      velocity="2" />
+	</joint>
+  <!-- Transmissions -->
   <transmission name="lift">
     <type>transmission_interface/SimpleTransmission</type>
@@ -435,5 +438,5 @@
     </actuator>
   </transmission>
-  <transmission name="mimic_lift">
+  <transmission name="mimic_lift1">
     <type>transmission_interface/SimpleTransmission</type>
     <joint name="lower_arm_joint"/>
@@ -443,5 +446,5 @@
     </actuator>
   </transmission>
-  <transmission name="mirror_lift">
+  <transmission name="mirror_lift2">
     <type>transmission_interface/SimpleTransmission</type>
     <joint name="metal_detector_arm_joint"/>
@@ -459,4 +462,5 @@
     </actuator>
   </transmission>
+  <!-- Gazebo mimic plugins -->
   <gazebo>
 	<plugin name="mimic_plugin1" filename="libgazebo_mimic_plugin.so">

File: urdf/fsr_husky_parts/front_cover.urdf.xacro (robot description, xacro)
@@ -27,14 +27,12 @@
 	xmlns:controller="http://playerstage.sourceforge.net/gazebo/xmlschema/#controller"
 	xmlns:interface="http://playerstage.sourceforge.net/gazebo/xmlschema/#interface"
-	xmlns:xacro="http://ros.org/wiki/xacro" name="husky_bridge">
-	<!-- Bridge -->
+	xmlns:xacro="http://ros.org/wiki/xacro" name="front_cover">
+	<!-- Front Cover -->
+  	<xacro:property name="scale_factor" value="0.001" />
 	<xacro:property name="husky_width" value="0.42" />
-	<xacro:property name="husky_heigh" value="0.245" />
-	<xacro:property name="scale_factor" value="0.001" />
-	<xacro:property name="bridge_height" value="0.385" />
-	<xacro:macro name="husky_bridge" params="parent x y z rx ry rz">
-		<link name="husky_bridge">
+	<xacro:macro name="front_cover" params="parent x y z rx ry rz">
+		<link name="front_cover">
 			<inertial>
-      				<origin xyz="1.3205E-08 -0.12511 0.1844" rpy="0 0 0" />
+      				<origin xyz="0 0 0.1844" rpy="0 0 0" />
      				 <mass value="0.41909" />
       				<inertia
@@ -47,26 +45,26 @@
     			</inertial>
 			<visual>
-      				<origin xyz="-0.31 ${-husky_width/2} ${-husky_heigh-bridge_height}" rpy="1.5708 0 1.5708" />
+      				<origin xyz="0 ${-husky_width/2-0.002} -0.10" rpy="1.5708 0 1.5708" />
       				<geometry>
-					<mesh filename="package://hratc2015_framework/models/fsr_husky_parts/bridge.STL" scale="${scale_factor} ${scale_factor} ${scale_factor}" />
+					<mesh filename="package://hratc2015_framework/models/fsr_husky_parts/front_cover.STL" scale="${scale_factor} ${scale_factor} ${scale_factor}" />
       				</geometry>
-      				<material name="Black" />
+      				<material name="Yellow" />
     			</visual>
 			<collision>
-      				<origin xyz="-0.31 ${-husky_width/2} ${-husky_heigh}" rpy="1.5708 0 1.5708" />
+      				<origin xyz="0 ${-husky_width/2-0.002} -0.10" rpy="1.5708 0 1.5708" />
       				<geometry>
-					<mesh filename="package://hratc2015_framework/models/fsr_husky_parts/bridge.STL" scale="${scale_factor} ${scale_factor} ${scale_factor}" />
+					<mesh filename="package://hratc2015_framework/models/fsr_husky_parts/front_cover.STL" scale="${scale_factor} ${scale_factor} ${scale_factor}" />
       				</geometry>
     			</collision>
 		</link>
-		<gazebo reference="husky_bridge">
-	        	<material>Gazebo/Black</material>
+		<gazebo reference="front_cover">
+	        	<material>Gazebo/Yellow</material>
 	        	<turnGravityOff>false</turnGravityOff>
     		</gazebo>
-		<joint name="joint_husky_bridge" type="fixed">
+		<joint name="joint_front_cover" type="fixed">
 			<parent link="${parent}"/>
-			<child link="husky_bridge"/>
-			<origin xyz="${x+0.31} ${y} ${z+bridge_height}" rpy="${rx} ${ry} ${rz}" />
+			<child link="front_cover"/>
+			<origin xyz="${x} ${y} ${z}" rpy="${rx} ${ry} ${rz}" />
 		</joint>
-  	</xacro:macro>
+	</xacro:macro>
 </robot>

File: urdf/fsr_husky_parts/pointgrey_flea3.urdf.xacro (robot description, xacro)
@@ -29,8 +29,8 @@
 	xmlns:xacro="http://ros.org/wiki/xacro" name="pointgrey_flea3">
 	<!-- PointGrey Flea 3 -->
-	<xacro:include filename="$(find hratc2015_framework)/urdf/fsr_husky_parts/common.xacro" />
-	<xacro:property name="base_x" value="0.040" />
-	<xacro:property name="base_y" value="0.150" />
-	<xacro:property name="base_z" value="0.015" />
+	<xacro:include filename="$(find hratc2014_framework)/urdf/fsr_husky_parts/common.xacro" />
+	<xacro:property name="base_x" value="0.001" />
+	<xacro:property name="base_y" value="0.001" />
+	<xacro:property name="base_z" value="0.001" />
  	<xacro:property name="standoff_length" value="0.100" />
 	<xacro:property name="standoff_radius" value="0.020" />

File: urdf/fsr_husky_parts/tim55x.urdf.xacro (robot description, xacro)
@@ -27,40 +27,42 @@
 	xmlns:controller="http://playerstage.sourceforge.net/gazebo/xmlschema/#controller"
 	xmlns:interface="http://playerstage.sourceforge.net/gazebo/xmlschema/#interface"
-	xmlns:xacro="http://ros.org/wiki/xacro" name="sick_lms100">
+	xmlns:xacro="http://ros.org/wiki/xacro" name="tim_55x">
 	<!-- SICK LMS100-->
 	<xacro:include filename="$(find hratc2015_framework)/urdf/fsr_husky_parts/common.xacro" />
+	<xacro:property name="scale_factor" value="0.001" />
 	<xacro:property name="laser_x" value="0.105" />
 	<xacro:property name="laser_y" value="0.102" />
 	<xacro:property name="laser_z" value="0.152" />
 	<xacro:property name="laser_mass" value="1.1" />
-	<xacro:macro name="sick_lms100" params="parent x y z rx ry rz">
-  		<link name="sick_lms100">
+	<xacro:macro name="tim_55x" params="parent x y z rx ry rz">
+  		<link name="tim_55x">
 			<xacro:box_inertial x="${laser_x}" y="${laser_y}" z="${laser_z}" mass="${laser_mass}" />
 			<visual>
-				<origin xyz="0 0 0" rpy="0 0 0" />
+				<origin xyz="-0.120 -0.075 -0.06246" rpy="-1.5708 -1.5708 0" />
 				<geometry>
-					<mesh filename="package://hratc2015_framework/models/fsr_husky_parts/sick_lms100.stl" />
+					<mesh filename="package://hratc2015_framework/models/fsr_husky_parts/tim55x.STL" scale="${scale_factor} ${scale_factor} ${scale_factor}" />
 				</geometry>
 				<material name="DarkGray" />
   			</visual>
     			<collision>
+				<origin xyz="-0.120 -0.075 -0.06246" rpy="-1.5708 -1.5708 0" />
       				<geometry>
-					<mesh filename="package://hratc2015_framework/models/fsr_husky_parts/sick_lms100.stl" />
+					<mesh filename="package://hratc2015_framework/models/fsr_husky_parts/tim55x.STL" scale="${scale_factor} ${scale_factor} ${scale_factor}" />
         				<!-- <box size="${laser_x} ${laser_y} ${laser_z}" /> -->
       				</geometry>
     			</collision>
   		</link>
-		<joint name="joint_sick_lms100" type="fixed">
+		<joint name="joint_tim_55x" type="fixed">
 			<parent link="${parent}"/>
-			<child link="sick_lms100"/>
-			<origin xyz="${x} ${y} ${z}" rpy="${rx} ${ry} ${rz}" />
+			<child link="tim_55x"/>
+			<origin xyz="${x} ${y} ${z+0.06246}" rpy="${rx} ${ry} ${rz}" />
 		</joint>
-		<gazebo reference="sick_lms100">
+		<gazebo reference="tim_55x">
 			<material>Gazebo/Grey</material>
 			<turnGravityOff>true</turnGravityOff>
-    			<sensor type="ray" name="sick_lms100">
+    			<sensor type="ray" name="tim_55x">
       				<pose>0 0 0 0 0 0</pose>
       				<visualize>false</visualize>
-     	 			<update_rate>40</update_rate>
+     	 			<update_rate>15</update_rate>
       				<ray>
         				<scan>
@@ -73,6 +75,6 @@
         				</scan>
         				<range>
-          					<min>0.10</min>
-          					<max>30.0</max>
+          					<min>0.05</min>
+          					<max>10.0</max>
           					<resolution>0.01</resolution>
         				</range>
@@ -85,5 +87,5 @@
       				<plugin name="gazebo_ros_laser" filename="libgazebo_ros_laser.so">
         				<topicName>scan</topicName>
-        				<frameName>sick_lms100</frameName>
+        				<frameName>tim_55x</frameName>
       				</plugin>
     			</sensor>

File: urdf/fsr_husky_parts/top_cover.urdf.xacro (robot description, xacro)
@@ -27,14 +27,12 @@
 	xmlns:controller="http://playerstage.sourceforge.net/gazebo/xmlschema/#controller"
 	xmlns:interface="http://playerstage.sourceforge.net/gazebo/xmlschema/#interface"
-	xmlns:xacro="http://ros.org/wiki/xacro" name="husky_bridge">
-	<!-- Bridge -->
+	xmlns:xacro="http://ros.org/wiki/xacro" name="top_cover">
+	<!-- Top Cover -->
+  	<xacro:property name="scale_factor" value="0.001" />
 	<xacro:property name="husky_width" value="0.42" />
-	<xacro:property name="husky_heigh" value="0.245" />
-	<xacro:property name="scale_factor" value="0.001" />
-	<xacro:property name="bridge_height" value="0.385" />
-	<xacro:macro name="husky_bridge" params="parent x y z rx ry rz">
-		<link name="husky_bridge">
+	<xacro:macro name="top_cover" params="parent x y z rx ry rz">
+		<link name="top_cover">
 			<inertial>
-      				<origin xyz="1.3205E-08 -0.12511 0.1844" rpy="0 0 0" />
+      				<origin xyz="0 0 0.1844" rpy="0 0 0" />
      				 <mass value="0.41909" />
       				<inertia
@@ -47,26 +45,26 @@
     			</inertial>
 			<visual>
-      				<origin xyz="-0.31 ${-husky_width/2} ${-husky_heigh-bridge_height}" rpy="1.5708 0 1.5708" />
+      				<origin xyz="0.07 ${-husky_width/2-0.0025} -0.10" rpy="1.5708 0 1.5708" />
       				<geometry>
-					<mesh filename="package://hratc2015_framework/models/fsr_husky_parts/bridge.STL" scale="${scale_factor} ${scale_factor} ${scale_factor}" />
+					<mesh filename="package://hratc2015_framework/models/fsr_husky_parts/top_cover.STL" scale="${scale_factor} ${scale_factor} ${scale_factor}" />
       				</geometry>
-      				<material name="Black" />
+      				<material name="Yellow" />
     			</visual>
 			<collision>
-      				<origin xyz="-0.31 ${-husky_width/2} ${-husky_heigh}" rpy="1.5708 0 1.5708" />
+      				<origin xyz="0.0 ${-husky_width/2-0.0025} -0.10" rpy="1.5708 0 1.5708" />
       				<geometry>
-					<mesh filename="package://hratc2015_framework/models/fsr_husky_parts/bridge.STL" scale="${scale_factor} ${scale_factor} ${scale_factor}" />
+					<mesh filename="package://hratc2015_framework/models/fsr_husky_parts/top_cover.STL" scale="${scale_factor} ${scale_factor} ${scale_factor}" />
       				</geometry>
     			</collision>
 		</link>
-		<gazebo reference="husky_bridge">
-	        	<material>Gazebo/Black</material>
+		<gazebo reference="top_cover">
+	        	<material>Gazebo/Yellow</material>
 	        	<turnGravityOff>false</turnGravityOff>
     		</gazebo>
-		<joint name="joint_husky_bridge" type="fixed">
+		<joint name="joint_top_cover" type="fixed">
 			<parent link="${parent}"/>
-			<child link="husky_bridge"/>
-			<origin xyz="${x+0.31} ${y} ${z+bridge_height}" rpy="${rx} ${ry} ${rz}" />
+			<child link="top_cover"/>
+			<origin xyz="${x} ${y} ${z}" rpy="${rx} ${ry} ${rz}" />
 		</joint>
-  	</xacro:macro>
+	</xacro:macro>
 </robot>
