Commit message: Update to the URDF model for the new Husky

File: urdf/husky.urdf.xacro (robot description, xacro)
@@ -46,11 +46,13 @@
     <xacro:include filename="$(find hratc2015_framework)/urdf/husky_parts/parts.urdf.xacro" />
     <xacro:include filename="$(find hratc2015_framework)/urdf/fsr_husky_parts/husky_bridge.urdf.xacro" />
-    <xacro:include filename="$(find hratc2015_framework)/urdf/fsr_husky_parts/sick_lms100.urdf.xacro" />
+    <xacro:include filename="$(find hratc2015_framework)/urdf/fsr_husky_parts/tim55x.urdf.xacro" />
     <xacro:include filename="$(find hratc2015_framework)/urdf/fsr_husky_parts/alfa_tube2h.urdf.xacro" />
     <xacro:include filename="$(find hratc2015_framework)/urdf/fsr_husky_parts/pointgrey_flea3.urdf.xacro" />
     <xacro:include filename="$(find hratc2015_framework)/urdf/fsr_husky_parts/gps_antenna.urdf.xacro" />
-    <xacro:include filename="$(find hratc2015_framework)/urdf/fsr_husky_parts/ptu_d46.urdf.xacro" />
+    <xacro:include filename="$(find hratc2015_framework)/urdf/fsr_husky_parts/tilt.urdf.xacro" />
     <xacro:include filename="$(find hratc2015_framework)/urdf/fsr_husky_parts/mti.urdf.xacro" />
     <xacro:include filename="$(find hratc2015_framework)/urdf/arm/fsr_husky_arm.urdf.xacro" />
+    <xacro:include filename="$(find hratc2015_framework)/urdf/fsr_husky_parts/front_cover.urdf.xacro" />
+    <xacro:include filename="$(find hratc2015_framework)/urdf/fsr_husky_parts/top_cover.urdf.xacro" />
     <!-- PROPERTY LIST -->
     <!--All units in m-kg-s-radians unit system -->
@@ -151,11 +153,4 @@
     </gazebo>
     <!-- Bumpers -->
-    <husky_part parent="base_footprint" name="front_bumper" mesh="bumper"
-          colour="DarkGray"
-          translateX="0.490" translateY="0.0" translateZ="${0.091 + wheel_x_size/2 - base_z_origin_to_wheel_origin}"
-          rotateX="0.0" rotateY="0.0" rotateZ="0.0"/>
-    <gazebo reference="base_footprint_front_bumper_part">
-        <material>Gazebo/FlatBlack</material>
-    </gazebo>
     <husky_part parent="base_footprint" name="rear_bumper" mesh="bumper"
           colour="DarkGray"
@@ -180,21 +175,24 @@
     <!-- FSR Husky Stuff -->
     <!-- BRIDGE macros -->
-    <husky_bridge prefix="front" parent="base_link" x="0.17" y="0" z="${base_z_size}" rx="0" ry="0" rz="0" />
-    <husky_bridge prefix="back" parent="base_link" x="-0.18" y="0" z="${base_z_size}" rx="0" ry="0" rz="0" />
+    <husky_bridge parent="base_link" x="-0.27" y="0" z="${base_z_size}" rx="0" ry="0" rz="0" />
+    <!-- Top cover macros -->
+    <top_cover parent="base_footprint" x="-0.18" y="0" z="${base_z_size}" rx="0" ry="0" rz="0" />
+    <!-- Front cover macros -->
+    <front_cover parent="base_footprint" x="0" y="0" z="${base_z_size}" rx="0" ry="0" rz="0" />
     <!-- MTi macro -->
-    <mti parent="back_husky_bridge" x="0" y="0" z="0.0" rx="0" ry="0" rz="0" />
+    <mti parent="husky_bridge" x="-0.10" y="0.17" z="-0.15" rx="1.57" ry="0" rz="0" />
     <!-- CAMERA macros -->
-    <pointgrey_flea3 prefix="right" parent="front_husky_bridge" base_offset="-0.13" camera_offset="-0.05" camera_r="0" camera_p="0" camera_y="0" />
-    <pointgrey_flea3 prefix="left" parent="front_husky_bridge" base_offset="0.13" camera_offset="0.05" camera_r="0" camera_p="0" camera_y="0" />
-    <!-- PTU-D46 macro -->
-    <ptu_d46 parent="front_husky_bridge" x="0" y="-0.025" z="0" rx="0" ry="0" rz="1.5708" />
-    <!-- SICK macro -->
-    <sick_lms100 parent="ptu_d46_tilt_link" x="0.0" y="0.13" z="0.11" rx="0.0" ry="-0.7854" rz="-1.5708" />
+    <pointgrey_flea3 prefix="right" parent="husky_bridge" base_offset="-0.145" camera_offset="-0.00" camera_r="0" camera_p="0" camera_y="0" />
+    <pointgrey_flea3 prefix="left" parent="husky_bridge" base_offset="0.145" camera_offset="0.00" camera_r="0" camera_p="0" camera_y="0" />
+    <!-- Tilt macro -->
+    <tilt parent="husky_bridge" x="0.055" y="0.0" z="0.029" rx="0" ry="0" rz="0" />
+    <!-- TIM macro -->
+    <tim_55x parent="tilt_link" x="0.015" y="0.0" z="-0.005" rx="0.0" ry="0" rz="0" />
     <!-- GPS macro -->
-    <gps_antenna parent="back_husky_bridge" x="0" y="0.17" z="0.0" rx="0" ry="0" rz="0" />
+    <gps_antenna parent="husky_bridge" x="0" y="-0.07" z="0.0" rx="0" ry="0" rz="0" />
     <!-- WiFi Antenna -->
-    <alfa_tube2h parent="back_husky_bridge" x="0" y="-0.17" z="0" rx="0" ry="0" rz="0" />
+    <alfa_tube2h parent="husky_bridge" x="-0.21" y="0.17" z="-0.38" rx="0" ry="0" rz="0" />
     <!-- FSR Husky De-mining Arm -->
-    <fsr_husky_arm parent="base_link" x="0.120" y="-0.15" z="${base_z_size}" rx="0" ry="0" rz="0" />
+    <fsr_husky_arm parent="base_link" x="0.0" y="0.0" z="0.0" rx="0" ry="0" rz="${M_PI/2}" />
     <gazebo>
       <plugin name="gazebo_ros_control" filename="libgazebo_ros_control.so">

Commit message: updated the position of the arm

File: urdf/arm/fsr_husky_arm.urdf.xacro (robot description, xacro)
@@ -134,5 +134,5 @@
 	<limit
       lower="-1.5708"
-      upper="3.14"
+      upper="3.06"
       effort="75"
       velocity="2" />
@@ -197,5 +197,5 @@
     <limit
       lower="-0.5236"
-      upper="0.5236"
+      upper="0.16"
       effort="35"
       velocity="2" />
@@ -219,6 +219,6 @@
     <visual>
       <origin
-        xyz="0 0 0"
-        rpy="0 0 0" />
+        xyz="0.0255 0.0026 -0.01050"
+        rpy="-1.865 -0.1 -1" />
       <geometry>
         <mesh
@@ -233,6 +233,6 @@
     <collision>
       <origin
-        xyz="0 0 0"
-        rpy="0 0 0" />
+        xyz="0.0255 0.0026 -0.01050"
+        rpy="-1.865 -0.1 -1" />
       <geometry>
         <mesh
@@ -253,5 +253,5 @@
       multiplier="-1" />
     <origin
-      xyz="-0.783340615005693 0.189233712627677 0.0344999999999998"
+      xyz="0.0 0.0344999999999998 0.8483340615005693"
       rpy="-1.5707963267949 1.140744854051 -1.26098072342103" />
     <parent
@@ -263,5 +263,5 @@
 	<limit
       lower="-0.5236"
-      upper="0.5236"
+      upper="0.16"
       effort="35"
       velocity="2" />
@@ -285,6 +285,6 @@
     <visual>
       <origin
-        xyz="0 0 0"
-        rpy="0 0 0" />
+        xyz="0.026 0 -0.29"
+        rpy="-1.9 -0.45 -1.45" />
       <geometry>
         <mesh
@@ -299,6 +299,6 @@
     <collision>
       <origin
-        xyz="0 0 0"
-        rpy="0 0 0" />
+        xyz="0.026 0 -0.29"
+        rpy="-1.9 -0.45 -1.45" />
       <geometry>
         <mesh
@@ -316,6 +316,6 @@
     type="fixed">
     <origin
-      xyz="0 0 0"
-      rpy="0 -2.7756E-17 -1.3878E-17" />
+      xyz="0.0350 -0.075 0.27"
+      rpy="0.350 0 0.42" /> -->
     <parent
       link="metal_detector_arm" />
@@ -334,5 +334,5 @@
   </link>
   <joint name="left_coil_joint" type="fixed">
-      <origin xyz="0.18 0 0" rpy="0 0 0" />
+      <origin xyz="0.18 -0.02 0.04" rpy="0 0 0" />
       <parent link="metal_detector_antenna"/>
       <child link="left_coil" />
@@ -347,5 +347,5 @@
   </link>
   <joint name="middle_coil_joint" type="fixed">
-      <origin xyz="0 0 0" rpy="0 0 0" />
+      <origin xyz="0 -0.02 0.04" rpy="0 0 0" />
       <parent link="metal_detector_antenna"/>
       <child link="middle_coil" />
@@ -360,5 +360,5 @@
   </link>
   <joint name="right_coil_joint" type="fixed">
-      <origin xyz="-0.18 0 0" rpy="0 0 0" />
+      <origin xyz="-0.18 -0.02 0.04" rpy="0 0 0" />
       <parent link="metal_detector_antenna"/>
       <child link="right_coil" />
@@ -425,5 +425,5 @@
     <limit
       lower="-0.5236"
-      upper="0.5236"
+      upper="0.16"
       effort="35"
       velocity="2" />

Commit message: Update do the URDF model

File: urdf/arm/fsr_husky_arm.urdf.xacro (robot description, xacro)
@@ -132,5 +132,5 @@
     <axis
       xyz="0 -1 0" />
-	<limit
+    <limit
       lower="-1.5708"
       upper="3.06"
@@ -262,6 +262,6 @@
       xyz="0.397068061333986 -0.865669276483222 -0.30488302416088" />
 	<limit
-      lower="-1.0"
-      upper="1.0"
+      lower="-0.5236"
+      upper="0.16"
       effort="35"
       velocity="2" />
@@ -432,5 +432,7 @@
   <transmission name="lift">
     <type>transmission_interface/SimpleTransmission</type>
-    <joint name="upper_arm_joint"/>
+    <joint name="upper_arm_joint">
+      <hardwareInterface>EffortJointInterface</hardwareInterface>
+    </joint>
     <actuator name="lift_motor">
       <hardwareInterface>EffortJointInterface</hardwareInterface>
@@ -440,5 +442,7 @@
   <transmission name="mimic_lift1">
     <type>transmission_interface/SimpleTransmission</type>
-    <joint name="lower_arm_joint"/>
+    <joint name="lower_arm_joint">
+      <hardwareInterface>EffortJointInterface</hardwareInterface>
+    </joint>
     <actuator name="mimic_lift_motor">
       <hardwareInterface>EffortJointInterface</hardwareInterface>
@@ -448,5 +452,7 @@
   <transmission name="mirror_lift2">
     <type>transmission_interface/SimpleTransmission</type>
-    <joint name="metal_detector_arm_joint"/>
+    <joint name="metal_detector_arm_joint">
+      <hardwareInterface>EffortJointInterface</hardwareInterface>
+    </joint>
     <actuator name="mirror_lift_motor">
       <hardwareInterface>EffortJointInterface</hardwareInterface>
@@ -456,5 +462,7 @@
   <transmission name="sweep">
     <type>transmission_interface/SimpleTransmission</type>
-    <joint name="arm_axel_joint"/>
+    <joint name="arm_axel_joint">
+      <hardwareInterface>EffortJointInterface</hardwareInterface>
+    </joint>
     <actuator name="sweep_motor">
       <hardwareInterface>EffortJointInterface</hardwareInterface>

File: urdf/husky.urdf.xacro (robot description, xacro)
@@ -68,12 +68,12 @@
     <property name="base_z_size" value="0.24750000" />
     <!--Weight of the base-->
-    <property name="base_mass" value="3.345489000" /> <!-- in kg-->
+    <property name="base_mass" value="33.45489000" /> <!-- in kg-->
     <!--Inertial values for the base at center of mass, aligned with coordinate system. Units are kg*m^2-->
-    <property name="base_ixx_com_cs" value="6.0216370" />
-    <property name="base_ixy_com_cs" value="0.0" />
-    <property name="base_ixz_com_cs" value="0.0" />
-    <property name="base_iyy_com_cs" value="17.3859574" />
-    <property name="base_iyz_com_cs" value="0.0" />
-    <property name="base_izz_com_cs" value="20.2955229" />
+    <property name="base_ixx_com_cs" value="0.60216370" />
+    <property name="base_ixy_com_cs" value="-0.02364198" />
+    <property name="base_ixz_com_cs" value="-0.11972132" />
+    <property name="base_iyy_com_cs" value="1.73859574" />
+    <property name="base_iyz_com_cs" value="-0.00154437" />
+    <property name="base_izz_com_cs" value="2.02955229" />
     <!-- BASE-FOOTPRINT -->
     <!-- base_footprint is a fictitious link(frame) that is on the ground right below base_link origin, navigation stack depends on this frame -->
@@ -181,5 +181,5 @@
     <front_cover parent="base_footprint" x="0" y="0" z="${base_z_size}" rx="0" ry="0" rz="0" />
     <!-- MTi macro -->
-    <mti parent="husky_bridge" x="-0.10" y="0.17" z="-0.15" rx="1.57" ry="0" rz="0" />
+    <mti parent="top_cover" x="0.2295" y="0.0" z="0.157" rx="0" ry="0" rz="0" />
     <!-- CAMERA macros -->
     <pointgrey_flea3 prefix="right" parent="husky_bridge" base_offset="-0.145" camera_offset="-0.00" camera_r="0" camera_p="0" camera_y="0" />

File: urdf/husky_parts/wheel.urdf.xacro (robot description, xacro)
@@ -89,5 +89,7 @@
 		<transmission name="joint_${fb}_${lr}_wheel_trans">
 			<type>transmission_interface/SimpleTransmission</type>
-			<joint name="joint_${fb}_${lr}_wheel" />
+			<joint name="joint_${fb}_${lr}_wheel" >
+			  <hardwareInterface>EffortJointInterface</hardwareInterface>
+			  </joint>
 			<actuator name="joint_${fb}_${lr}_wheel_motor">
 			  <hardwareInterface>EffortJointInterface</hardwareInterface>
