Commit message: Robot update (metal detector and bridge are now attached to the URDF model)

File: description/urdf/p3at_sonar.urdf.xacro (robot description, xacro)
@@ -1,6 +1,6 @@
 <?xml version="1.0"?>
 <robot xmlns:xacro="http://www.ros.org/wiki/xacro">
-    <xacro:include filename="$(find p3at_phi_framework)/description/urdf/common.xacro" />
-    <xacro:include filename="$(find p3at_phi_framework)/description/urdf/sonar_sensor.urdf.xacro" />
+    <xacro:include filename="$(find hratc2017_framework)/description/urdf/common.xacro" />
+    <xacro:include filename="$(find hratc2017_framework)/description/urdf/sonar_sensor.urdf.xacro" />
 	<xacro:property name="update_rate" value="10" />
 	<xacro:property name="min_range" value="0.15" />

File: description/urdf/pioneer3at.urdf.xacro (robot description, xacro)
@@ -6,8 +6,13 @@
 name="pioneer3at">
 <!-- Included URDF/XACRO Files -->
-<xacro:include filename="$(find p3at_phi_framework)/description/urdf/common.xacro" />
-<xacro:include filename="$(find p3at_phi_framework)/description/urdf/sick_lms100.urdf.xacro" />
-<xacro:include filename="$(find p3at_phi_framework)/description/urdf/pointgrey_flea3.urdf.xacro" />
-<xacro:include filename="$(find p3at_phi_framework)/description/urdf/p3at_sonar.urdf.xacro" />
+<xacro:include filename="$(find hratc2017_framework)/description/urdf/common.xacro" />
+<xacro:include filename="$(find hratc2017_framework)/description/urdf/sick_lms100.urdf.xacro" />
+<xacro:include filename="$(find hratc2017_framework)/description/urdf/sick_tim55x.urdf.xacro" />
+<xacro:include filename="$(find hratc2017_framework)/description/urdf/sick_tim.urdf.xacro" />
+<xacro:include filename="$(find hratc2017_framework)/description/urdf/pointgrey_flea3.urdf.xacro" />
+<xacro:include filename="$(find hratc2017_framework)/description/urdf/p3at_sonar.urdf.xacro" />
+<xacro:include filename="$(find hratc2017_framework)/description/urdf/gps_antenna.urdf.xacro" />
+<xacro:include filename="$(find metal_detector_msgs)/model/gazebo/metal_detector.urdf.xacro" />
+<xacro:include filename="$(find hratc2017_robot)/model/gazebo/Bridge.urdf.xacro" />
 <!-- Chassis -->
     <link name="base_link">
@@ -27,5 +32,5 @@
             <origin xyz="0 0 0.177" rpy="0 0 0"/>
             <geometry name="pioneer_geom">
-                <mesh filename="package://p3at_phi_framework/description/p3at_meshes/chassis.stl"/>
+                <mesh filename="package://hratc2017_framework/description/p3at_meshes/chassis.stl"/>
             </geometry>
             <material name="ChassisRed">
@@ -36,5 +41,5 @@
             <origin xyz="0 0 0.177" rpy="0 0 0"/>
             <geometry>
-                <mesh filename="package://p3at_phi_framework/description/p3at_meshes/chassis.stl"/>
+                <mesh filename="package://hratc2017_framework/description/p3at_meshes/chassis.stl"/>
             </geometry>
         </collision>
@@ -55,5 +60,5 @@
             <origin xyz="0 0 0" rpy="0 0 0"/>
             <geometry name="pioneer_geom">
-                <mesh filename="package://p3at_phi_framework/description/p3at_meshes/top.stl"/>
+                <mesh filename="package://hratc2017_framework/description/p3at_meshes/top.stl"/>
             </geometry>
             <material name="TopBlack">
@@ -78,24 +83,24 @@
 <!-- Front + Back Sonar -->
     <link name="front_sonar">
-        <inertial>
-            <mass value="0.1"/>
-            <origin xyz="0 0 0"/>
-            <inertia ixx="1.0" ixy="0.0" ixz="0.0" iyy="1.0" iyz="0.0" izz="1.0"/>
-        </inertial>
-        <visual name="base_visual">
-            <origin xyz="0 0 0" rpy="0 0 0"/>
-            <geometry name="pioneer_geom">
-                <mesh filename="package://p3at_phi_framework/description/p3at_meshes/front_sonar.stl"/>
-            </geometry>
-            <material name="SonarYellow">
-                <color rgba="0.715 0.583 0.210 1.0"/>
-            </material>
-        </visual>
-        <collision>
-            <origin xyz="0 0 0" rpy="0 0 0"/>
-            <geometry>
-                <box size="0 0 0"/>
-            </geometry>
-        </collision>
+<!--        <inertial>-->
+<!--            <mass value="0.1"/>    -->
+<!--            <origin xyz="0 0 0"/>-->
+<!--            <inertia ixx="1.0" ixy="0.0" ixz="0.0" iyy="1.0" iyz="0.0" izz="1.0"/>-->
+<!--        </inertial>-->
+<!--        <visual name="base_visual">-->
+<!--            <origin xyz="0 0 0" rpy="0 0 0"/>-->
+<!--            <geometry name="pioneer_geom">-->
+<!--                <mesh filename="package://hratc2017_framework/description/p3at_meshes/front_sonar.stl"/>-->
+<!--            </geometry>-->
+<!--            <material name="SonarYellow">-->
+<!--                <color rgba="0.715 0.583 0.210 1.0"/>-->
+<!--            </material>-->
+<!--        </visual>-->
+<!--        <collision>-->
+<!--            <origin xyz="0 0 0" rpy="0 0 0"/>-->
+<!--            <geometry>-->
+<!--                <box size="0 0 0"/>-->
+<!--            </geometry>-->
+<!--        </collision>-->
     </link>
     <gazebo reference="front_sonar">
@@ -108,24 +113,24 @@
     </joint>
     <link name="back_sonar">
-        <inertial>
-            <mass value="0.1"/>
-            <origin xyz="0 0 0"/>
-            <inertia ixx="1.0" ixy="0.0" ixz="0.0" iyy="1.0" iyz="0.0" izz="1.0"/>
-        </inertial>
-        <visual name="base_visual">
-            <origin xyz="0 0 0" rpy="0 0 0"/>
-            <geometry name="pioneer_geom">
-                <mesh filename="package://p3at_phi_framework/description/p3at_meshes/back_sonar.stl"/>
-            </geometry>
-            <material name="SonarYellow">
-                <color rgba="0.715 0.583 0.210 1.0"/>
-            </material>
-        </visual>
-        <collision>
-            <origin xyz="0 0 0" rpy="0 0 0"/>
-            <geometry>
-                <box size="0 0 0"/>
-            </geometry>
-        </collision>
+<!--        <inertial>-->
+<!--            <mass value="0.1"/>    -->
+<!--            <origin xyz="0 0 0"/>-->
+<!--            <inertia ixx="1.0" ixy="0.0" ixz="0.0" iyy="1.0" iyz="0.0" izz="1.0"/>-->
+<!--        </inertial>-->
+<!--        <visual name="base_visual">-->
+<!--            <origin xyz="0 0 0" rpy="0 0 0"/>-->
+<!--            <geometry name="pioneer_geom">-->
+<!--                <mesh filename="package://hratc2017_framework/description/p3at_meshes/back_sonar.stl"/>-->
+<!--            </geometry>-->
+<!--            <material name="SonarYellow">-->
+<!--                <color rgba="0.715 0.583 0.210 1.0"/>-->
+<!--            </material>-->
+<!--        </visual>-->
+<!--        <collision>-->
+<!--            <origin xyz="0 0 0" rpy="0 0 0"/>-->
+<!--            <geometry>-->
+<!--                <box size="0 0 0"/>-->
+<!--            </geometry>-->
+<!--        </collision>-->
     </link>
     <gazebo reference="back_sonar">
@@ -148,5 +153,5 @@
             <origin xyz="0 0 0" rpy="0 0 0"/>
             <geometry name="pioneer_geom">
-                <mesh filename="package://p3at_phi_framework/description/p3at_meshes/axle.stl"/>
+                <mesh filename="package://hratc2017_framework/description/p3at_meshes/axle.stl"/>
             </geometry>
             <material name="AxleGrey">
@@ -178,5 +183,5 @@
             <origin xyz="0 0 0" rpy="0 0 0"/>
             <geometry name="pioneer_geom">
-                <mesh filename="package://p3at_phi_framework/description/p3at_meshes/${side}_hubcap.stl"/>
+                <mesh filename="package://hratc2017_framework/description/p3at_meshes/${side}_hubcap.stl"/>
             </geometry>
             <material name="HubcapYellow">
@@ -208,5 +213,5 @@
             <origin xyz="0 0 0" rpy="0 0 0"/>
             <geometry name="pioneer_geom">
-                <mesh filename="package://p3at_phi_framework/description/p3at_meshes/wheel.stl"/>
+                <mesh filename="package://hratc2017_framework/description/p3at_meshes/wheel.stl"/>
             </geometry>
             <material name="WheelBlack">
@@ -217,5 +222,5 @@
             <origin xyz="0 0 0" rpy="${-3.1415927/2} 0 0"/>
             <geometry>
-                <!--mesh filename="package://p3at_phi_framework/description/p3at_meshes/wheel.stl"/-->
+                <!--mesh filename="package://hratc2017_framework/description/p3at_meshes/wheel.stl"/-->
                 <cylinder radius="0.111" length="0.075"/>
             </geometry>
@@ -244,5 +249,5 @@
             <origin xyz="0 0 0" rpy="0 0 0"/>
             <geometry name="pioneer_geom">
-                <mesh filename="package://p3at_phi_framework/description/p3at_meshes/axle.stl"/>
+                <mesh filename="package://hratc2017_framework/description/p3at_meshes/axle.stl"/>
             </geometry>
             <material name="AxleGrey">
@@ -253,5 +258,5 @@
             <origin xyz="0 0 0" rpy="0 0 0"/>
             <geometry>
-                <mesh filename="package://p3at_phi_framework/description/p3at_meshes/axle.stl"/>
+                <mesh filename="package://hratc2017_framework/description/p3at_meshes/axle.stl"/>
             </geometry>
         </collision>
@@ -274,5 +279,5 @@
             <origin xyz="0 0 0" rpy="0 0 0"/>
             <geometry name="pioneer_geom">
-                <mesh filename="package://p3at_phi_framework/description/p3at_meshes/${side}_hubcap.stl"/>
+                <mesh filename="package://hratc2017_framework/description/p3at_meshes/${side}_hubcap.stl"/>
             </geometry>
             <material name="HubcapYellow"/>
@@ -281,5 +286,5 @@
             <origin xyz="0 0 0" rpy="0 0 0"/>
             <geometry>
-                <mesh filename="package://p3at_phi_framework/description/p3at_meshes/${side}_hubcap.stl"/>
+                <mesh filename="package://hratc2017_framework/description/p3at_meshes/${side}_hubcap.stl"/>
             </geometry>
         </collision>
@@ -302,5 +307,5 @@
             <origin xyz="0 0 0" rpy="0 0 0"/>
             <geometry name="pioneer_geom">
-                <mesh filename="package://p3at_phi_framework/description/p3at_meshes/wheel.stl"/>
+                <mesh filename="package://hratc2017_framework/description/p3at_meshes/wheel.stl"/>
             </geometry>
             <material name="WheelBlack"/>
@@ -309,5 +314,5 @@
             <origin xyz="0 0 0" rpy="${-3.1415927/2} 0 0"/>
             <geometry>
-            <!--mesh filename="package://p3at_phi_framework/description/p3at_meshes/wheel.stl"/-->
+            <!--mesh filename="package://hratc2017_framework/description/p3at_meshes/wheel.stl"/-->
             <cylinder radius="0.111" length="0.075"/>
             </geometry>
@@ -385,6 +390,18 @@
 <xacro:p3at_drive_side side="right" reflect="-1"/>
 <xacro:p3at_gazebo_ext/>
+<!-- metal detector macro -->
+<metal_detector parent="front_sonar">
+    <origin xyz="0.0 0.09 -0.16" rpy="0 0 ${-90*M_PI/180}"/>
+</metal_detector>
+<!-- robot bridge macro -->
+<robot_bridge parent="top_plate">
+    <origin xyz="-0.14 -0.14 0.0" rpy="0 0 0"/>
+</robot_bridge>
 <!-- SICK macro -->
-<sick_lms100 parent="base_link" x="0.2" y="0.0" z="0.4" rx="0.0" ry="${0*M_PI/180}" rz="0.0" />
+<!--<sick_lms100 parent="robot_bridge_top" x="0.15" y="0.05" z="0.12" rx="0.0" ry="0.0" rz="${90*M_PI/180}" />-->
+<sick_tim_55x parent="robot_bridge_top" x="0.095" y="0.0" z="0.07" rx="${-90*M_PI/180}" ry="0.0" rz="0.0" />
+<!--<sick_tim310 name="laser" ros_topic="scan" parent="base_link" x="0.2" y="0.0" z="0.4" rx="0.0" ry="${0*M_PI/180}" rz="0.0" />-->
+<!-- GPS macro -->
+<gps_antenna parent="robot_bridge_top" x="0" y="-0.07" z="0.0" rx="0" ry="0" rz="0" />
 <!-- CAMERA macros -->
 <!--<pointgrey_flea3 prefix="right" parent="base_link" base_offset="-0.3" camera_offset="-0.05" camera_r="0" camera_p="0" camera_y="0" />-->

File: description/urdf/sick_tim55x.urdf.xacro (robot description, xacro)
@@ -1,5 +1,4 @@
 <?xml version="1.0"?>
 <!--
-Copyright (c) 2016, Renan Maffei, Phi Robotics Reseach Group, INF - UFRGS
 Copyright (c) 2013, Goncalo Cabrita, ISR University of Coimbra
 All rights reserved.
@@ -28,40 +27,42 @@
 	xmlns:controller="http://playerstage.sourceforge.net/gazebo/xmlschema/#controller"
 	xmlns:interface="http://playerstage.sourceforge.net/gazebo/xmlschema/#interface"
-	xmlns:xacro="http://ros.org/wiki/xacro" name="sick_lms100">
-	<!-- SICK LMS100-->
+	xmlns:xacro="http://ros.org/wiki/xacro" name="tim_55x">
 	<xacro:include filename="$(find hratc2017_framework)/description/urdf/common.xacro" />
+	<xacro:property name="scale_factor" value="0.001" />
 	<xacro:property name="laser_x" value="0.105" />
 	<xacro:property name="laser_y" value="0.102" />
 	<xacro:property name="laser_z" value="0.152" />
 	<xacro:property name="laser_mass" value="1.1" />
-	<xacro:macro name="sick_lms100" params="parent x y z rx ry rz">
-  		<link name="sick_lms100">
-            <xacro:box_inertial x="${laser_x}" y="${laser_y}" z="${laser_z}" mass="${laser_mass}" />
-            <visual>
-                <origin xyz="0 0 0" rpy="0 0 0" />
-                <geometry>
-                    <mesh filename="package://hratc2017_framework/description/sensors_meshes/sick_lms100.stl" />
-                </geometry>
-                <material name="DarkGray" />
-            </visual>
-            <collision>
-                <geometry>
-                    <mesh filename="package://hratc2017_framework/description/sensors_meshes/sick_lms100.stl" />
-                    <!-- <box size="${laser_x} ${laser_y} ${laser_z}" /> -->
-                </geometry>
-            </collision>
-        </link>
-		<joint name="joint_sick_lms100" type="fixed">
-			<parent link="${parent}"/>
-			<child link="sick_lms100"/>
-			<origin xyz="${x} ${y} ${z}" rpy="${rx} ${ry} ${rz}" />
+	<xacro:macro name="sick_tim_55x" params="parent x y z rx ry rz">
+  		<link name="tim_55x">
+			<xacro:box_inertial x="${laser_x}" y="${laser_y}" z="${laser_z}" mass="${laser_mass}" />
+			<visual>
+				<origin xyz="-0.121 -0.075 -0.064" rpy="0 -1.5708 -1.5708" />
+				<geometry>
+					<mesh filename="package://hratc2017_framework/description/sensors_meshes/sick_tim55x.STL" scale="${scale_factor} ${scale_factor} ${scale_factor}" />
+				</geometry>
+				<material name="DarkGray" />
+  			</visual>
+    			<collision>
+				<origin xyz="-0.121 -0.075 -0.064" rpy="0 -1.5708 -1.5708" />
+      				<geometry>
+					<mesh filename="package://hratc2017_framework/description/sensors_meshes/sick_tim55x.STL" scale="${scale_factor} ${scale_factor} ${scale_factor}" />
+        				<!-- <box size="${laser_x} ${laser_y} ${laser_z}" /> -->
+      				</geometry>
+    			</collision>
+  		</link>
+		<joint name="joint_tim_55x" type="fixed">
+		  <origin xyz="${x+0.054558} ${y+0.022286} ${z}" rpy="${rx+1.5708} ${ry+2.8361E-16} ${rz+1.6214}" />
+		  <parent link="${parent}"/>
+		  <child link="tim_55x" />
+		  <axis xyz="0 0 0" />
 		</joint>
-		<gazebo reference="sick_lms100">
+		<gazebo reference="tim_55x">
 			<material>Gazebo/Grey</material>
 			<turnGravityOff>true</turnGravityOff>
-    			<sensor type="ray" name="sick_lms100">
+    			<sensor type="ray" name="tim_55x">
       				<pose>0 0 0 0 0 0</pose>
       				<visualize>false</visualize>
-     	 			<update_rate>40</update_rate>
+     	 			<update_rate>15</update_rate>
       				<ray>
         				<scan>
@@ -74,6 +75,6 @@
         				</scan>
         				<range>
-          					<min>0.10</min>
-          					<max>30.0</max>
+          					<min>0.05</min>
+          					<max>10.0</max>
           					<resolution>0.01</resolution>
         				</range>
@@ -86,5 +87,5 @@
       				<plugin name="gazebo_ros_laser" filename="libgazebo_ros_laser.so">
         				<topicName>scan</topicName>
-        				<frameName>sick_lms100</frameName>
+        				<frameName>tim_55x</frameName>
       				</plugin>
     			</sensor>

File: description/urdf/sonar_sensor.urdf.xacro (robot description, xacro)
@@ -17,5 +17,5 @@
 <!--        <origin xyz="0 0 0" rpy="0 0 0" />-->
 <!--        <geometry>-->
-<!--          <mesh filename="package://p3at_phi_framework/description/sensors_meshes/max_sonar_ez4.dae"/>-->
+<!--          <mesh filename="package://hratc2017_framework/description/sensors_meshes/max_sonar_ez4.dae"/>-->
 <!--        </geometry>-->
 <!--      </visual>-->
