Commit message: Update of some urdf files

File: description/urdf/pioneer3at.urdf (robot description, URDF)
Before this commit: robot pioneer3at, 16 links, 15 joints
Links:
- link back_sonar: geometry collision box size=0 0 0; visual mesh filename=package://hratc2017_framework/description/p3at_meshes/back_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
- link base_link: geometry collision mesh filename=package://hratc2017_framework/description/p3at_meshes/chass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; visual mesh filename=package://hratc2017_framework/description/p3at_meshes/chass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
- link front_sonar: geometry collision box size=0 0 0; visual mesh filename=package://hratc2017_framework/description/p3at_meshes/front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
- link p3at_back_left_axle: geometry collision mesh filename=package://hratc2017_framework/description/p3at_meshes/axle.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; visual mesh filename=package://hratc2017_framework/description/p3at_meshes/axle.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
- link p3at_back_left_hub: geometry collision mesh filename=package://hratc2017_framework/description/p3at_meshes/left_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; visual mesh filename=package://hratc2017_framework/description/p3at_meshes/left_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
- link p3at_back_left_wheel: geometry collision cylinder length=0.075 radius=0.111; visual mesh filename=package://hratc2017_framework/description/p3at_meshes/wheel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
- link p3at_back_right_axle: geometry collision mesh filename=package://hratc2017_framework/description/p3at_meshes/axle.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; visual mesh filename=package://hratc2017_framework/description/p3at_meshes/axle.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
- link p3at_back_right_hub: geometry collision mesh filename=package://hratc2017_framework/description/p3at_meshes/right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; visual mesh filename=package://hratc2017_framework/description/p3at_meshes/right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
- link p3at_back_right_wheel: geometry collision cylinder length=0.075 radius=0.111; visual mesh filename=package://hratc2017_framework/description/p3at_meshes/wheel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
- link p3at_front_left_axle: geometry collision box size=0 0 0; visual mesh filename=package://hratc2017_framework/description/p3at_meshes/axle.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
- link p3at_front_left_hub: geometry collision box size=0 0 0; visual mesh filename=package://hratc2017_framework/description/p3at_meshes/left_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
- link p3at_front_left_wheel: geometry collision cylinder length=0.075 radius=0.111; visual mesh filename=package://hratc2017_framework/description/p3at_meshes/wheel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
- link p3at_front_right_axle: geometry collision box size=0 0 0; visual mesh filename=package://hratc2017_framework/description/p3at_meshes/axle.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
- link p3at_front_right_hub: geometry collision box size=0 0 0; visual mesh filename=package://hratc2017_framework/description/p3at_meshes/right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
- link p3at_front_right_wheel: geometry collision cylinder length=0.075 radius=0.111; visual mesh filename=package://hratc2017_framework/description/p3at_meshes/wheel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
- link top_plate: geometry collision box size=0 0 0; visual mesh filename=package://hratc2017_framework/description/p3at_meshes/top.s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

File: description/urdf/pioneer3at_ptu.urdf.xacro (robot description, xacro)
@@ -6,6 +6,6 @@
 name="pioneer3at">
 <!-- Included URDF/XACRO Files -->
-<xacro:include filename="$(find p3at_phi_framework)/description/urdf/sick_lms100.urdf.xacro" />
-<xacro:include filename="$(find p3at_phi_framework)/description/urdf/ptu_d46.urdf.xacro" />
+<xacro:include filename="$(find hratc2017_framework)/description/urdf/sick_lms100.urdf.xacro" />
+<xacro:include filename="$(find hratc2017_framework)/description/urdf/ptu_d46.urdf.xacro" />
 <!-- Chassis -->
     <link name="base_link">
@@ -25,5 +25,5 @@
             <origin xyz="0 0 0.177" rpy="0 0 0"/>
             <geometry name="pioneer_geom">
-                <mesh filename="package://p3at_phi_framework/description/p3at_meshes/chassis.stl"/>
+                <mesh filename="package://hratc2017_framework/description/p3at_meshes/chassis.stl"/>
             </geometry>
             <material name="ChassisRed">
@@ -34,5 +34,5 @@
             <origin xyz="0 0 0.177" rpy="0 0 0"/>
             <geometry>
-                <mesh filename="package://p3at_phi_framework/description/p3at_meshes/chassis.stl"/>
+                <mesh filename="package://hratc2017_framework/description/p3at_meshes/chassis.stl"/>
             </geometry>
         </collision>
@@ -53,5 +53,5 @@
             <origin xyz="0 0 0" rpy="0 0 0"/>
             <geometry name="pioneer_geom">
-                <mesh filename="package://p3at_phi_framework/description/p3at_meshes/top.stl"/>
+                <mesh filename="package://hratc2017_framework/description/p3at_meshes/top.stl"/>
             </geometry>
             <material name="TopBlack">
@@ -84,5 +84,5 @@
             <origin xyz="0 0 0" rpy="0 0 0"/>
             <geometry name="pioneer_geom">
-                <mesh filename="package://p3at_phi_framework/description/p3at_meshes/front_sonar.stl"/>
+                <mesh filename="package://hratc2017_framework/description/p3at_meshes/front_sonar.stl"/>
             </geometry>
             <material name="SonarYellow">
@@ -114,5 +114,5 @@
             <origin xyz="0 0 0" rpy="0 0 0"/>
             <geometry name="pioneer_geom">
-                <mesh filename="package://p3at_phi_framework/description/p3at_meshes/back_sonar.stl"/>
+                <mesh filename="package://hratc2017_framework/description/p3at_meshes/back_sonar.stl"/>
             </geometry>
             <material name="SonarYellow">
@@ -146,5 +146,5 @@
             <origin xyz="0 0 0" rpy="0 0 0"/>
             <geometry name="pioneer_geom">
-                <mesh filename="package://p3at_phi_framework/description/p3at_meshes/axle.stl"/>
+                <mesh filename="package://hratc2017_framework/description/p3at_meshes/axle.stl"/>
             </geometry>
             <material name="AxleGrey">
@@ -176,5 +176,5 @@
             <origin xyz="0 0 0" rpy="0 0 0"/>
             <geometry name="pioneer_geom">
-                <mesh filename="package://p3at_phi_framework/description/p3at_meshes/${side}_hubcap.stl"/>
+                <mesh filename="package://hratc2017_framework/description/p3at_meshes/${side}_hubcap.stl"/>
             </geometry>
             <material name="HubcapYellow">
@@ -206,5 +206,5 @@
             <origin xyz="0 0 0" rpy="0 0 0"/>
             <geometry name="pioneer_geom">
-                <mesh filename="package://p3at_phi_framework/description/p3at_meshes/wheel.stl"/>
+                <mesh filename="package://hratc2017_framework/description/p3at_meshes/wheel.stl"/>
             </geometry>
             <material name="WheelBlack">
@@ -215,5 +215,5 @@
             <origin xyz="0 0 0" rpy="${-3.1415927/2} 0 0"/>
             <geometry>
-                <!--mesh filename="package://p3at_phi_framework/description/p3at_meshes/wheel.stl"/-->
+                <!--mesh filename="package://hratc2017_framework/description/p3at_meshes/wheel.stl"/-->
                 <cylinder radius="0.111" length="0.075"/>
             </geometry>
@@ -242,5 +242,5 @@
             <origin xyz="0 0 0" rpy="0 0 0"/>
             <geometry name="pioneer_geom">
-                <mesh filename="package://p3at_phi_framework/description/p3at_meshes/axle.stl"/>
+                <mesh filename="package://hratc2017_framework/description/p3at_meshes/axle.stl"/>
             </geometry>
             <material name="AxleGrey">
@@ -251,5 +251,5 @@
             <origin xyz="0 0 0" rpy="0 0 0"/>
             <geometry>
-                <mesh filename="package://p3at_phi_framework/description/p3at_meshes/axle.stl"/>
+                <mesh filename="package://hratc2017_framework/description/p3at_meshes/axle.stl"/>
             </geometry>
         </collision>
@@ -272,5 +272,5 @@
             <origin xyz="0 0 0" rpy="0 0 0"/>
             <geometry name="pioneer_geom">
-                <mesh filename="package://p3at_phi_framework/description/p3at_meshes/${side}_hubcap.stl"/>
+                <mesh filename="package://hratc2017_framework/description/p3at_meshes/${side}_hubcap.stl"/>
             </geometry>
             <material name="HubcapYellow"/>
@@ -279,5 +279,5 @@
             <origin xyz="0 0 0" rpy="0 0 0"/>
             <geometry>
-                <mesh filename="package://p3at_phi_framework/description/p3at_meshes/${side}_hubcap.stl"/>
+                <mesh filename="package://hratc2017_framework/description/p3at_meshes/${side}_hubcap.stl"/>
             </geometry>
         </collision>
@@ -300,5 +300,5 @@
             <origin xyz="0 0 0" rpy="0 0 0"/>
             <geometry name="pioneer_geom">
-                <mesh filename="package://p3at_phi_framework/description/p3at_meshes/wheel.stl"/>
+                <mesh filename="package://hratc2017_framework/description/p3at_meshes/wheel.stl"/>
             </geometry>
             <material name="WheelBlack"/>
@@ -307,5 +307,5 @@
             <origin xyz="0 0 0" rpy="${-3.1415927/2} 0 0"/>
             <geometry>
-            <!--mesh filename="package://p3at_phi_framework/description/p3at_meshes/wheel.stl"/-->
+            <!--mesh filename="package://hratc2017_framework/description/p3at_meshes/wheel.stl"/-->
             <cylinder radius="0.111" length="0.075"/>
             </geometry>

File: description/urdf/pioneer3at_sonar.urdf.xacro (robot description, xacro)
@@ -6,8 +6,8 @@
 name="pioneer3at">
 <!-- Included URDF/XACRO Files -->
-<xacro:include filename="$(find p3at_phi_framework)/description/urdf/common.xacro" />
-<xacro:include filename="$(find p3at_phi_framework)/description/urdf/sick_lms100.urdf.xacro" />
-<xacro:include filename="$(find p3at_phi_framework)/description/urdf/pointgrey_flea3.urdf.xacro" />
-<xacro:include filename="$(find p3at_phi_framework)/description/urdf/p3at_sonar.urdf.xacro" />
+<xacro:include filename="$(find hratc2017_framework)/description/urdf/common.xacro" />
+<xacro:include filename="$(find hratc2017_framework)/description/urdf/sick_lms100.urdf.xacro" />
+<xacro:include filename="$(find hratc2017_framework)/description/urdf/pointgrey_flea3.urdf.xacro" />
+<xacro:include filename="$(find hratc2017_framework)/description/urdf/p3at_sonar.urdf.xacro" />
 <!-- Chassis -->
     <link name="base_link">
@@ -27,5 +27,5 @@
             <origin xyz="0 0 0.177" rpy="0 0 0"/>
             <geometry name="pioneer_geom">
-                <mesh filename="package://p3at_phi_framework/description/p3at_meshes/chassis.stl"/>
+                <mesh filename="package://hratc2017_framework/description/p3at_meshes/chassis.stl"/>
             </geometry>
             <material name="ChassisRed">
@@ -36,5 +36,5 @@
             <origin xyz="0 0 0.177" rpy="0 0 0"/>
             <geometry>
-                <mesh filename="package://p3at_phi_framework/description/p3at_meshes/chassis.stl"/>
+                <mesh filename="package://hratc2017_framework/description/p3at_meshes/chassis.stl"/>
             </geometry>
         </collision>
@@ -55,5 +55,5 @@
             <origin xyz="0 0 0" rpy="0 0 0"/>
             <geometry name="pioneer_geom">
-                <mesh filename="package://p3at_phi_framework/description/p3at_meshes/top.stl"/>
+                <mesh filename="package://hratc2017_framework/description/p3at_meshes/top.stl"/>
             </geometry>
             <material name="TopBlack">
@@ -86,5 +86,5 @@
             <origin xyz="0 0 0" rpy="0 0 0"/>
             <geometry name="pioneer_geom">
-                <mesh filename="package://p3at_phi_framework/description/p3at_meshes/front_sonar.stl"/>
+                <mesh filename="package://hratc2017_framework/description/p3at_meshes/front_sonar.stl"/>
             </geometry>
             <material name="SonarYellow">
@@ -116,5 +116,5 @@
             <origin xyz="0 0 0" rpy="0 0 0"/>
             <geometry name="pioneer_geom">
-                <mesh filename="package://p3at_phi_framework/description/p3at_meshes/back_sonar.stl"/>
+                <mesh filename="package://hratc2017_framework/description/p3at_meshes/back_sonar.stl"/>
             </geometry>
             <material name="SonarYellow">
@@ -148,5 +148,5 @@
             <origin xyz="0 0 0" rpy="0 0 0"/>
             <geometry name="pioneer_geom">
-                <mesh filename="package://p3at_phi_framework/description/p3at_meshes/axle.stl"/>
+                <mesh filename="package://hratc2017_framework/description/p3at_meshes/axle.stl"/>
             </geometry>
             <material name="AxleGrey">
@@ -178,5 +178,5 @@
             <origin xyz="0 0 0" rpy="0 0 0"/>
             <geometry name="pioneer_geom">
-                <mesh filename="package://p3at_phi_framework/description/p3at_meshes/${side}_hubcap.stl"/>
+                <mesh filename="package://hratc2017_framework/description/p3at_meshes/${side}_hubcap.stl"/>
             </geometry>
             <material name="HubcapYellow">
@@ -208,5 +208,5 @@
             <origin xyz="0 0 0" rpy="0 0 0"/>
             <geometry name="pioneer_geom">
-                <mesh filename="package://p3at_phi_framework/description/p3at_meshes/wheel.stl"/>
+                <mesh filename="package://hratc2017_framework/description/p3at_meshes/wheel.stl"/>
             </geometry>
             <material name="WheelBlack">
@@ -217,5 +217,5 @@
             <origin xyz="0 0 0" rpy="${-3.1415927/2} 0 0"/>
             <geometry>
-                <!--mesh filename="package://p3at_phi_framework/description/p3at_meshes/wheel.stl"/-->
+                <!--mesh filename="package://hratc2017_framework/description/p3at_meshes/wheel.stl"/-->
                 <cylinder radius="0.111" length="0.075"/>
             </geometry>
@@ -244,5 +244,5 @@
             <origin xyz="0 0 0" rpy="0 0 0"/>
             <geometry name="pioneer_geom">
-                <mesh filename="package://p3at_phi_framework/description/p3at_meshes/axle.stl"/>
+                <mesh filename="package://hratc2017_framework/description/p3at_meshes/axle.stl"/>
             </geometry>
             <material name="AxleGrey">
@@ -253,5 +253,5 @@
             <origin xyz="0 0 0" rpy="0 0 0"/>
             <geometry>
-                <mesh filename="package://p3at_phi_framework/description/p3at_meshes/axle.stl"/>
+                <mesh filename="package://hratc2017_framework/description/p3at_meshes/axle.stl"/>
             </geometry>
         </collision>
@@ -274,5 +274,5 @@
             <origin xyz="0 0 0" rpy="0 0 0"/>
             <geometry name="pioneer_geom">
-                <mesh filename="package://p3at_phi_framework/description/p3at_meshes/${side}_hubcap.stl"/>
+                <mesh filename="package://hratc2017_framework/description/p3at_meshes/${side}_hubcap.stl"/>
             </geometry>
             <material name="HubcapYellow"/>
@@ -281,5 +281,5 @@
             <origin xyz="0 0 0" rpy="0 0 0"/>
             <geometry>
-                <mesh filename="package://p3at_phi_framework/description/p3at_meshes/${side}_hubcap.stl"/>
+                <mesh filename="package://hratc2017_framework/description/p3at_meshes/${side}_hubcap.stl"/>
             </geometry>
         </collision>
@@ -302,5 +302,5 @@
             <origin xyz="0 0 0" rpy="0 0 0"/>
             <geometry name="pioneer_geom">
-                <mesh filename="package://p3at_phi_framework/description/p3at_meshes/wheel.stl"/>
+                <mesh filename="package://hratc2017_framework/description/p3at_meshes/wheel.stl"/>
             </geometry>
             <material name="WheelBlack"/>
@@ -309,5 +309,5 @@
             <origin xyz="0 0 0" rpy="${-3.1415927/2} 0 0"/>
             <geometry>
-            <!--mesh filename="package://p3at_phi_framework/description/p3at_meshes/wheel.stl"/-->
+            <!--mesh filename="package://hratc2017_framework/description/p3at_meshes/wheel.stl"/-->
             <cylinder radius="0.111" length="0.075"/>
             </geometry>

File: description/urdf/pointgrey_flea3.urdf.xacro (robot description, xacro)
@@ -30,5 +30,5 @@
 	xmlns:xacro="http://ros.org/wiki/xacro" name="pointgrey_flea3">
 	<!-- PointGrey Flea 3 -->
-	<xacro:include filename="$(find p3at_phi_framework)/description/urdf/common.xacro" />
+	<xacro:include filename="$(find hratc2017_framework)/description/urdf/common.xacro" />
 	<xacro:property name="base_x" value="0.040" />
 	<xacro:property name="base_y" value="0.150" />

File: description/urdf/ptu_d46.urdf.xacro (robot description, xacro)
@@ -40,5 +40,5 @@
                 <origin xyz="0 0 0" rpy="0 0 0" />
                 <geometry>
-                    <mesh filename="package://p3at_phi_framework/description/sensors_meshes/ptu_d46_base_link.stl" />
+                    <mesh filename="package://hratc2017_framework/description/sensors_meshes/ptu_d46_base_link.stl" />
                 </geometry>
                 <material name="DarkGray" />
@@ -47,5 +47,5 @@
                 <origin xyz="0 0 0" rpy="0 0 0" />
                 <geometry>
-                    <mesh filename="package://p3at_phi_framework/description/sensors_meshes/ptu_d46_base_link.stl" />
+                    <mesh filename="package://hratc2017_framework/description/sensors_meshes/ptu_d46_base_link.stl" />
                 </geometry>
             </collision>
@@ -69,5 +69,5 @@
                 <origin xyz="0 0 0" rpy="0 0 0" />
                 <geometry>
-                    <mesh filename="package://p3at_phi_framework/description/sensors_meshes/ptu_d46_pan_link.stl" />
+                    <mesh filename="package://hratc2017_framework/description/sensors_meshes/ptu_d46_pan_link.stl" />
                 </geometry>
                 <material name="DarkGray" />
@@ -76,5 +76,5 @@
                 <origin xyz="0 0 0" rpy="0 0 0" />
                 <geometry>
-                    <mesh filename="package://p3at_phi_framework/description/sensors_meshes/ptu_d46_pan_link.stl" />
+                    <mesh filename="package://hratc2017_framework/description/sensors_meshes/ptu_d46_pan_link.stl" />
                 </geometry>
             </collision>
@@ -101,5 +101,5 @@
                 <origin xyz="0 0 0" rpy="0 0 0" />
                 <geometry>
-                    <mesh filename="package://p3at_phi_framework/description/sensors_meshes/ptu_d46_tilt_link.stl" />
+                    <mesh filename="package://hratc2017_framework/description/sensors_meshes/ptu_d46_tilt_link.stl" />
                 </geometry>
                 <material name="DarkGray" />
@@ -108,5 +108,5 @@
                 <origin xyz="0 0 0" rpy="0 0 0" />
                 <geometry>
-                    <mesh filename="package://p3at_phi_framework/description/sensors_meshes/ptu_d46_tilt_link.stl" />
+                    <mesh filename="package://hratc2017_framework/description/sensors_meshes/ptu_d46_tilt_link.stl" />
                 </geometry>
             </collision>
