Commit message: Major changes in the robot description; Added 2nd laser range finder, imu and robot_pose_ekf

File: description/urdf/gps_antenna.urdf.xacro (robot description, xacro)
@@ -34,32 +34,30 @@
 	<xacro:property name="antenna_length" value="0.45" />
 	<xacro:property name="antenna_radius" value="0.008" />
-	<xacro:macro name="gps_antenna" params="parent x y z rx ry rz">
+    <xacro:macro name="gps_antenna" params="parent x y z rx ry rz">
   		<link name="gps_antenna">
-    			<inertial>
-      				<origin xyz="0.035 1.27350000005198E-07 0.084899" rpy="0 0 0" />
-      				<mass value="0.28321" />
-      				<inertia
-        				ixx="0.000632544028273332"
-        				ixy="-4.4923388876054E-20"
-        				ixz="1.07422508310795E-20"
-        				iyy="1.26609361466704E-09"
-        				iyz="-0.000632544028277925"
-        				izz="-1.26609361462022E-09" />
-    			</inertial>
-    			<visual>
-      				<origin xyz="-0.035 0 0" rpy="1.5708 0 0" />
-      				<geometry>
-					<mesh filename="package://hratc2017_framework/description/sensors_meshes/gps_antenna.stl" />
-      				</geometry>
-      				<material name="White">
-        				<color rgba="1 1 1 1"/>
-      				</material>
-    			</visual>
-    			<collision>
-      				<origin xyz="-0.035 0 0" rpy="1.5708 0 0" />
-      				<geometry>
-					<mesh filename="package://hratc2017_framework/description/sensors_meshes/gps_antenna.stl" />
-     			 	</geometry>
-    			</collision>
+            <inertial>
+                <origin xyz="0.035 1.27350000005198E-07 0.084899" rpy="0 0 0" />
+                <mass value="0.28321" />
+                <inertia
+                ixx="0.000632544028273332"
+                ixy="-4.4923388876054E-20"
+                ixz="1.07422508310795E-20"
+                iyy="1.26609361466704E-09"
+                iyz="-0.000632544028277925"
+                izz="-1.26609361462022E-09" />
+            </inertial>
+            <visual>
+                <origin xyz="0 0 0" rpy="0 0 0" />
+                <geometry>
+                    <box size="0.045 0.042 0.0135"/>
+                </geometry>
+                <material name="Black"/>
+            </visual>
+            <collision>
+                <origin xyz="0 0 0" rpy="0 0 0" />
+                <geometry>
+                    <box size="0.045 0.042 0.0135"/>
+                </geometry>
+            </collision>
   		</link>
 		<joint name="gps_antenna_joint" type="fixed">
@@ -69,21 +67,25 @@
 		</joint>
 		<gazebo reference="gps_antenna">
-        		<material>Gazebo/White</material>
-        		<turnGravityOff>false</turnGravityOff>
+            <material>Gazebo/Black</material>
+            <turnGravityOff>false</turnGravityOff>
 		</gazebo>
-		<gazebo>
-			<plugin name="gazebo_ros_gps" filename="libgazebo_gps_plugin.so">
-			  <updateRate>4.0</updateRate>
-			  <bodyName>gps_antenna</bodyName>
-			  <frameId>gps_antenna</frameId>
-			  <topicName>/gps/fix</topicName>
-			  <velocityTopicName>/gps/fix_velocity</velocityTopicName>
-			  <offset>0 0 0</offset>
-			  <drift>0.001 0.001 0.001</drift>
-			  <gaussianNoise>0.01 0.01 0.01</gaussianNoise>
-			  <velocityDrift>0 0 0</velocityDrift>
-			  <velocityGaussianNoise>0.05 0.05 0.05</velocityGaussianNoise>
-			</plugin>
-    		</gazebo>
+        <gazebo>
+            <plugin name="gazebo_ros_gps" filename="libhector_gazebo_ros_gps.so">
+                <updateRate>4.0</updateRate>
+                <bodyName>gps_antenna</bodyName>
+                <frameId>gps_antenna</frameId>
+                <topicName>/gps/fix</topicName>
+                <velocityTopicName>/gps/fix_velocity</velocityTopicName>
+                <referenceLatitude>40.184680128</referenceLatitude>
+                <referenceLongitude>-8.414337443</referenceLongitude>
+<!--                <referenceHeading>0</referenceHeading>-->
+                <referenceAltitude>119.4501</referenceAltitude>
+                <offset>0 0 0</offset>
+                <drift>0.001 0.001 0.001</drift>
+                <gaussianNoise>0.01 0.01 0.01</gaussianNoise>
+                <velocityDrift>0 0 0</velocityDrift>
+                <velocityGaussianNoise>0.05 0.05 0.05</velocityGaussianNoise>
+            </plugin>
+        </gazebo>
 	</xacro:macro>
 </robot>

File: description/urdf/pioneer3at.urdf.xacro (robot description, xacro)
@@ -10,4 +10,6 @@
 <xacro:include filename="$(find hratc2017_framework)/description/urdf/sick_tim55x.urdf.xacro" />
 <xacro:include filename="$(find hratc2017_framework)/description/urdf/sick_tim.urdf.xacro" />
+<xacro:include filename="$(find hratc2017_framework)/description/urdf/hokuyo.urdf.xacro" />
+<xacro:include filename="$(find hratc2017_framework)/description/urdf/mti.urdf.xacro" />
 <xacro:include filename="$(find hratc2017_framework)/description/urdf/pointgrey_flea3.urdf.xacro" />
 <xacro:include filename="$(find hratc2017_framework)/description/urdf/p3at_sonar.urdf.xacro" />
@@ -15,4 +17,29 @@
 <xacro:include filename="$(find metal_detector_msgs)/model/gazebo/metal_detector.urdf.xacro" />
 <xacro:include filename="$(find hratc2017_robot)/model/gazebo/Bridge.urdf.xacro" />
+    <!-- BASE-FOOTPRINT -->
+    <!-- base_footprint is a fictitious link(frame) that is on the ground right below base_link origin, navigation stack depends on this frame -->
+    <link name="base_footprint">
+        <!--<inertial>
+            <mass value="0.0001" />
+            <origin xyz="0 0 0" />
+            <inertia ixx="0.0001" ixy="0.0" ixz="0.0"
+                iyy="0.0001" iyz="0.0"
+                izz="0.0001" />
+	      </inertial>-->
+        <visual>
+            <origin xyz="0 0 0" rpy="0 0 0" />
+            <geometry>
+                <box size="0.001 0.001 0.001" />
+            </geometry>
+        </visual>
+    </link>
+    <gazebo reference="base_footprint">
+        <turnGravityOff>false</turnGravityOff>
+    </gazebo>
+    <joint name="base_footprint_joint" type="fixed">
+		<origin xyz="0 0 0" rpy="0 0 0" />
+        <parent link="base_footprint"/>
+        <child link="base_link" />
+    </joint>
 <!-- Chassis -->
     <link name="base_link">
@@ -402,6 +429,10 @@
 <sick_tim_55x parent="robot_bridge_top" x="0.095" y="0.0" z="0.07" rx="${-90*M_PI/180}" ry="0.0" rz="0.0" />
 <!--<sick_tim310 name="laser" ros_topic="scan" parent="base_link" x="0.2" y="0.0" z="0.4" rx="0.0" ry="${0*M_PI/180}" rz="0.0" />-->
+<!-- Hokuyo macro -->
+<sensor_hokuyo parent="robot_bridge_box" x="0.12" y="0.14" z="0.22" rx="${0*M_PI/180}" ry="${(90-55)*M_PI/180}" rz="${0*M_PI/180}" />
 <!-- GPS macro -->
-<gps_antenna parent="robot_bridge_top" x="0" y="-0.07" z="0.0" rx="0" ry="0" rz="0" />
+<gps_antenna parent="robot_bridge_top" x="0.25" y="0.02" z="0.01" rx="0" ry="0" rz="0" />
+<!-- IMU macro -->
+<mti parent="robot_bridge_top" x="0.05" y="0.02" z="0.005" rx="0" ry="0" rz="0" />
 <!-- CAMERA macros -->
 <!--<pointgrey_flea3 prefix="right" parent="base_link" base_offset="-0.3" camera_offset="-0.05" camera_r="0" camera_p="0" camera_y="0" />-->

File: description/urdf/sick_tim55x.urdf.xacro (robot description, xacro)
@@ -68,8 +68,8 @@
         				<scan>
           					<horizontal>
-            						<samples>720</samples>
-            						<resolution>1</resolution>
-            						<min_angle>-1.570796</min_angle>
-            						<max_angle>1.570796</max_angle>
+        						<samples>720</samples>
+        						<resolution>1</resolution>
+        						<min_angle>-1.570796</min_angle>
+        						<max_angle>1.570796</max_angle>
           					</horizontal>
         				</scan>

Commit message: Cleaning of files no longer used.

File: description/urdf/gps_antenna.urdf.xacro (robot description, xacro)
@@ -82,7 +82,7 @@
                 <referenceAltitude>10</referenceAltitude>
                 <offset>0 0 0</offset>
-                <drift>0.00 0.00 0.00</drift>
+                <drift>0.001 0.001 0.001</drift>
                 <gaussianNoise>0.05 0.05 0.05</gaussianNoise>
-                <velocityDrift>0.01 0.05 0.05</velocityDrift>
+                <velocityDrift>0.001 0.001 0.001</velocityDrift>
                 <velocityGaussianNoise>0.5 0.5 0.5</velocityGaussianNoise>
 <!--                <drift>0.001 0.001 0.001</drift>-->

File: description/urdf/pioneer3at.urdf.xacro (robot description, xacro)
@@ -7,11 +7,7 @@
 <!-- Included URDF/XACRO Files -->
 <xacro:include filename="$(find hratc2017_framework)/description/urdf/common.xacro" />
-<xacro:include filename="$(find hratc2017_framework)/description/urdf/sick_lms100.urdf.xacro" />
 <xacro:include filename="$(find hratc2017_framework)/description/urdf/sick_tim55x.urdf.xacro" />
-<xacro:include filename="$(find hratc2017_framework)/description/urdf/sick_tim.urdf.xacro" />
 <xacro:include filename="$(find hratc2017_framework)/description/urdf/hokuyo.urdf.xacro" />
 <xacro:include filename="$(find hratc2017_framework)/description/urdf/mti.urdf.xacro" />
-<xacro:include filename="$(find hratc2017_framework)/description/urdf/pointgrey_flea3.urdf.xacro" />
-<xacro:include filename="$(find hratc2017_framework)/description/urdf/p3at_sonar.urdf.xacro" />
 <xacro:include filename="$(find hratc2017_framework)/description/urdf/gps_antenna.urdf.xacro" />
 <xacro:include filename="$(find metal_detector_msgs)/model/gazebo/metal_detector.urdf.xacro" />
@@ -426,7 +422,5 @@
 </robot_bridge>
 <!-- SICK macro -->
-<!--<sick_lms100 parent="robot_bridge_top" x="0.15" y="0.05" z="0.12" rx="0.0" ry="0.0" rz="${90*M_PI/180}" />-->
 <sick_tim_55x parent="robot_bridge_top" x="0.095" y="0.0" z="0.07" rx="${-90*M_PI/180}" ry="0.0" rz="0.0" />
-<!--<sick_tim310 name="laser" ros_topic="scan" parent="base_link" x="0.2" y="0.0" z="0.4" rx="0.0" ry="${0*M_PI/180}" rz="0.0" />-->
 <!-- Hokuyo macro -->
 <sensor_hokuyo parent="Hokuyo_joint" x="0.01" y="0.08" z="0.01" rx="${-90*M_PI/180}" ry="${0*M_PI/180}" rz="${0*M_PI/180}" />
@@ -435,13 +429,3 @@
 <!-- IMU macro -->
 <mti parent="robot_bridge_top" x="0.05" y="0.02" z="0.005" rx="${0*M_PI/180}" ry="${0*M_PI/180}" rz="${0*M_PI/180}" />
-<!-- CAMERA macros -->
-<!--<pointgrey_flea3 prefix="right" parent="base_link" base_offset="-0.3" camera_offset="-0.05" camera_r="0" camera_p="0" camera_y="0" />-->
-<!--<pointgrey_flea3 prefix="left" parent="base_link" base_offset="0.13" camera_offset="0.05" camera_r="0" camera_p="0" camera_y="0" />-->
-<!-- SONAR macros -->
-<!--<p3at_sonar prefix="front" parent="front_sonar">-->
-<!--    <origin xyz="0.0 0.0 0.0" rpy="0 0 0"/>-->
-<!--</p3at_sonar>-->
-<!--<p3at_sonar prefix="back" parent="back_sonar">-->
-<!--    <origin xyz="0.0 0.0 0.0" rpy="0 0 ${180*M_PI/180}"/>-->
-<!--</p3at_sonar>-->
 </robot>

Commit message: updated framework package

File: description/urdf/gps_antenna.urdf.xacro (robot description, xacro)
@@ -77,13 +77,17 @@
                 <topicName>/gps/fix</topicName>
                 <velocityTopicName>/gps/fix_velocity</velocityTopicName>
-                <referenceLatitude>40.184680128</referenceLatitude>
-                <referenceLongitude>-8.414337443</referenceLongitude>
+                <referenceLatitude>-30.06022459407145675</referenceLatitude>
+                <referenceLongitude>-51.173913575780311191</referenceLongitude>
                 <referenceHeading>90</referenceHeading>
-                <referenceAltitude>119.4501</referenceAltitude>
+                <referenceAltitude>10</referenceAltitude>
                 <offset>0 0 0</offset>
                 <drift>0.001 0.001 0.001</drift>
-                <gaussianNoise>0.01 0.01 0.01</gaussianNoise>
-                <velocityDrift>0 0 0</velocityDrift>
-                <velocityGaussianNoise>0.05 0.05 0.05</velocityGaussianNoise>
+                <gaussianNoise>0.05 0.05 0.05</gaussianNoise>
+                <velocityDrift>0.001 0.001 0.001</velocityDrift>
+                <velocityGaussianNoise>0.5 0.5 0.5</velocityGaussianNoise>
+<!--                <drift>0.001 0.001 0.001</drift>-->
+<!--                <gaussianNoise>0.01 0.01 0.01</gaussianNoise>-->
+<!--                <velocityDrift>0 0 0</velocityDrift>-->
+<!--                <velocityGaussianNoise>0.05 0.05 0.05</velocityGaussianNoise>-->
             </plugin>
         </gazebo>

File: description/urdf/mti.urdf.xacro (robot description, xacro)
@@ -60,5 +60,5 @@
             <plugin name="gazebo_ros_imu" filename="libgazebo_ros_imu.so">
                 <alwaysOn>true</alwaysOn>
-                <bodyName>base_footprint</bodyName>
+                <bodyName>base_link</bodyName>
                 <topicName>/imu/data</topicName>
                 <serviceName>imu_service</serviceName>

File: description/urdf/pioneer3at.urdf.xacro (robot description, xacro)
@@ -7,39 +7,10 @@
 <!-- Included URDF/XACRO Files -->
 <xacro:include filename="$(find hratc2017_framework)/description/urdf/common.xacro" />
-<xacro:include filename="$(find hratc2017_framework)/description/urdf/sick_lms100.urdf.xacro" />
 <xacro:include filename="$(find hratc2017_framework)/description/urdf/sick_tim55x.urdf.xacro" />
-<xacro:include filename="$(find hratc2017_framework)/description/urdf/sick_tim.urdf.xacro" />
 <xacro:include filename="$(find hratc2017_framework)/description/urdf/hokuyo.urdf.xacro" />
 <xacro:include filename="$(find hratc2017_framework)/description/urdf/mti.urdf.xacro" />
-<xacro:include filename="$(find hratc2017_framework)/description/urdf/pointgrey_flea3.urdf.xacro" />
-<xacro:include filename="$(find hratc2017_framework)/description/urdf/p3at_sonar.urdf.xacro" />
 <xacro:include filename="$(find hratc2017_framework)/description/urdf/gps_antenna.urdf.xacro" />
 <xacro:include filename="$(find metal_detector_msgs)/model/gazebo/metal_detector.urdf.xacro" />
 <xacro:include filename="$(find hratc2017_robot)/model/gazebo/Bridge.urdf.xacro" />
-    <!-- BASE-FOOTPRINT -->
-    <!-- base_footprint is a fictitious link(frame) that is on the ground right below base_link origin, navigation stack depends on this frame -->
-    <link name="base_footprint">
-        <!--<inertial>
-            <mass value="0.0001" />
-            <origin xyz="0 0 0" />
-            <inertia ixx="0.0001" ixy="0.0" ixz="0.0"
-                iyy="0.0001" iyz="0.0"
-                izz="0.0001" />
-	      </inertial>-->
-        <visual>
-            <origin xyz="0 0 0" rpy="0 0 0" />
-            <geometry>
-                <box size="0.001 0.001 0.001" />
-            </geometry>
-        </visual>
-    </link>
-    <gazebo reference="base_footprint">
-        <turnGravityOff>false</turnGravityOff>
-    </gazebo>
-    <joint name="base_footprint_joint" type="fixed">
-		<origin xyz="0 0 0" rpy="0 0 0" />
-        <parent link="base_footprint"/>
-        <child link="base_link" />
-    </joint>
 <!-- Chassis -->
     <link name="base_link">
@@ -426,7 +397,5 @@
 </robot_bridge>
 <!-- SICK macro -->
-<!--<sick_lms100 parent="robot_bridge_top" x="0.15" y="0.05" z="0.12" rx="0.0" ry="0.0" rz="${90*M_PI/180}" />-->
 <sick_tim_55x parent="robot_bridge_top" x="0.095" y="0.0" z="0.07" rx="${-90*M_PI/180}" ry="0.0" rz="0.0" />
-<!--<sick_tim310 name="laser" ros_topic="scan" parent="base_link" x="0.2" y="0.0" z="0.4" rx="0.0" ry="${0*M_PI/180}" rz="0.0" />-->
 <!-- Hokuyo macro -->
 <sensor_hokuyo parent="Hokuyo_joint" x="0.01" y="0.08" z="0.01" rx="${-90*M_PI/180}" ry="${0*M_PI/180}" rz="${0*M_PI/180}" />
@@ -435,13 +404,3 @@
 <!-- IMU macro -->
 <mti parent="robot_bridge_top" x="0.05" y="0.02" z="0.005" rx="${0*M_PI/180}" ry="${0*M_PI/180}" rz="${0*M_PI/180}" />
-<!-- CAMERA macros -->
-<!--<pointgrey_flea3 prefix="right" parent="base_link" base_offset="-0.3" camera_offset="-0.05" camera_r="0" camera_p="0" camera_y="0" />-->
-<!--<pointgrey_flea3 prefix="left" parent="base_link" base_offset="0.13" camera_offset="0.05" camera_r="0" camera_p="0" camera_y="0" />-->
-<!-- SONAR macros -->
-<!--<p3at_sonar prefix="front" parent="front_sonar">-->
-<!--    <origin xyz="0.0 0.0 0.0" rpy="0 0 0"/>-->
-<!--</p3at_sonar>-->
-<!--<p3at_sonar prefix="back" parent="back_sonar">-->
-<!--    <origin xyz="0.0 0.0 0.0" rpy="0 0 ${180*M_PI/180}"/>-->
-<!--</p3at_sonar>-->
 </robot>
